Commit message: Fixed gazebo simulation
- Fixed urdf files (wrong joint name in trasmission)
- Fixed iiwas_control.launch
- Fixed Gazebo launch file

File: iiwas_description/urdf/iiwa.transmission.xacro (robot description, xacro)
@@ -5,5 +5,5 @@
       <robotNamespace>/${robot_name}</robotNamespace>
       <type>transmission_interface/SimpleTransmission</type>
-      <joint name="${robot_name}_SFE">
+      <joint name="${robot_name}_joint_1">
 	    <hardwareInterface>${hardware_interface}</hardwareInterface>
       </joint>
@@ -16,5 +16,5 @@
       <robotNamespace>/${robot_name}</robotNamespace>
       <type>transmission_interface/SimpleTransmission</type>
-      <joint name="${robot_name}_SAA">
+      <joint name="${robot_name}_joint_2">
 	    <hardwareInterface>${hardware_interface}</hardwareInterface>
       </joint>
@@ -27,5 +27,5 @@
       <robotNamespace>/${robot_name}</robotNamespace>
       <type>transmission_interface/SimpleTransmission</type>
-      <joint name="${robot_name}_HR">
+      <joint name="${robot_name}_joint_3">
 	    <hardwareInterface>${hardware_interface}</hardwareInterface>
       </joint>
@@ -38,5 +38,5 @@
       <robotNamespace>/${robot_name}</robotNamespace>
       <type>transmission_interface/SimpleTransmission</type>
-      <joint name="${robot_name}_EB">
+      <joint name="${robot_name}_joint_4">
 	    <hardwareInterface>${hardware_interface}</hardwareInterface>
       </joint>
@@ -49,5 +49,5 @@
       <robotNamespace>/${robot_name}</robotNamespace>
       <type>transmission_interface/SimpleTransmission</type>
-      <joint name="${robot_name}_WR">
+      <joint name="${robot_name}_joint_5">
 	    <hardwareInterface>${hardware_interface}</hardwareInterface>
       </joint>
@@ -60,5 +60,5 @@
       <robotNamespace>/${robot_name}</robotNamespace>
       <type>transmission_interface/SimpleTransmission</type>
-      <joint name="${robot_name}_WFE">
+      <joint name="${robot_name}_joint_6">
 	    <hardwareInterface>${hardware_interface}</hardwareInterface>
       </joint>
@@ -71,5 +71,5 @@
       <robotNamespace>/${robot_name}</robotNamespace>
       <type>transmission_interface/SimpleTransmission</type>
-      <joint name="${robot_name}_WAA">
+      <joint name="${robot_name}_joint_7">
 	    <hardwareInterface>${hardware_interface}</hardwareInterface>
       </joint>

File: iiwas_description/urdf/iiwa14.xacro (robot description, xacro)
@@ -48,5 +48,4 @@
     </link>
     <!-- joint between link_0 and link_1 -->
-    <!--<joint name="${robot_name}_SFE" type="revolute">-->
     <joint name="${robot_name}_joint_1" type="revolute">
       <parent link="${robot_name}_link_0"/>
@@ -87,5 +86,4 @@
     </link>
     <!-- joint between link_1 and link_2 -->
-    <!--<joint name="${robot_name}_SAA" type="revolute">-->
     <joint name="${robot_name}_joint_2" type="revolute">
       <parent link="${robot_name}_link_1"/>
@@ -126,5 +124,4 @@
     </link>
     <!-- joint between link_2 and link_3 -->
-    <!--<joint name="${robot_name}_HR" type="revolute">-->
     <joint name="${robot_name}_joint_3" type="revolute">
       <parent link="${robot_name}_link_2"/>
@@ -165,5 +162,4 @@
     </link>
     <!-- joint between link_3 and link_4 -->
-    <!--<joint name="${robot_name}_EB" type="revolute">-->
     <joint name="${robot_name}_joint_4" type="revolute">
       <parent link="${robot_name}_link_3"/>
@@ -204,5 +200,4 @@
     </link>
     <!-- joint between link_4 and link_5 -->
-    <!--<joint name="${robot_name}_WR" type="revolute">-->
     <joint name="${robot_name}_joint_5" type="revolute">
       <parent link="${robot_name}_link_4"/>
@@ -243,5 +238,4 @@
     </link>
     <!-- joint between link_5 and link_6 -->
-    <!--<joint name="${robot_name}_WFE" type="revolute">-->
     <joint name="${robot_name}_joint_6" type="revolute">
       <parent link="${robot_name}_link_5"/>
@@ -282,5 +276,4 @@
     </link>
     <!-- joint between link_6 and link_7 -->
-    <!--<joint name="${robot_name}_WAA" type="revolute">-->
     <joint name="${robot_name}_joint_7" type="revolute">
       <parent link="${robot_name}_link_6"/>
