Commit message: Add iiwas_pybullet package, fix issues with gazebo
- use true simulation velocity
- consider options of erp and cfm
- refactor some variables
- add iiwas_pybullet package (controller needs to be tuned)
- increase the damping of urdf
- tune the controller parameter of simulation

File: iiwas_description/urdf/iiwa.gazebo.xacro (robot description, xacro)
@@ -59,7 +59,28 @@
     </gazebo>
     <!-- Link7 -->
-    <gazebo reference="${robot_name}_joint_ee">
-      <preserveFixedJoint>1</preserveFixedJoint>
-    </gazebo>
+<!--    <gazebo reference="${robot_name}_joint_ee">-->
+<!--      <preserveFixedJoint>1</preserveFixedJoint>-->
+<!--    </gazebo>-->
+<!--    <gazebo reference="${robot_name}_joint_1">-->
+<!--      <implicitSpringDamper>true</implicitSpringDamper>-->
+<!--    </gazebo>-->
+<!--    <gazebo reference="${robot_name}_joint_2">-->
+<!--      <implicitSpringDamper>true</implicitSpringDamper>-->
+<!--    </gazebo>-->
+<!--    <gazebo reference="${robot_name}_joint_3">-->
+<!--      <implicitSpringDamper>true</implicitSpringDamper>-->
+<!--    </gazebo>-->
+<!--    <gazebo reference="${robot_name}_joint_4">-->
+<!--      <implicitSpringDamper>true</implicitSpringDamper>-->
+<!--    </gazebo>-->
+<!--    <gazebo reference="${robot_name}_joint_5">-->
+<!--      <implicitSpringDamper>true</implicitSpringDamper>-->
+<!--    </gazebo>-->
+<!--    <gazebo reference="${robot_name}_joint_6">-->
+<!--      <implicitSpringDamper>true</implicitSpringDamper>-->
+<!--    </gazebo>-->
+<!--    <gazebo reference="${robot_name}_joint_7">-->
+<!--      <implicitSpringDamper>true</implicitSpringDamper>-->
+<!--    </gazebo>-->
   </xacro:macro>
 </robot>

File: iiwas_description/urdf/iiwa14.xacro (robot description, xacro)
@@ -182,5 +182,5 @@
       <xacro:unless value="${dynamics_parameter == 'eth'}">
         <!-- Identified -->
-        <dynamics damping="0.031758" friction="0.213255"/>
+        <dynamics damping="0.1" friction="0.213255"/>
       </xacro:unless>
     </joint>
@@ -300,5 +300,5 @@
       <xacro:unless value="${dynamics_parameter == 'eth'}">
         <!-- Identified -->
-        <dynamics damping="0.058755" friction="0.536120"/>
+        <dynamics damping="0.1" friction="0.536120"/>
       </xacro:unless>
     </joint>
@@ -359,5 +359,5 @@
       <xacro:unless value="${dynamics_parameter == 'eth'}">
         <!-- Identified -->
-		<dynamics damping="0.009696" friction="0.212718"/>
+		<dynamics damping="0.1" friction="0.212718"/>
       </xacro:unless>
     </joint>
@@ -418,5 +418,5 @@
       <xacro:unless value="${dynamics_parameter == 'eth'}">
         <!-- Identified -->
-		<dynamics damping="0.001000" friction="0.337016"/>
+		<dynamics damping="0.1" friction="0.337016"/>
       </xacro:unless>
     </joint>
