Commit message: set back the joint velocity limit of urdf

File: iiwas_description/urdf/iiwa14.xacro (robot description, xacro)
@@ -11,6 +11,4 @@
   <xacro:property name="safety_controller_k_vel" value="10" />
   <xacro:property name="joint_damping" value="0.5" />
-  <xacro:property name="max_effort" value="300"/>
-  <xacro:property name="max_velocity" value="1.309"/>
   <xacro:macro name="iiwa14" params="parent hardware_interface robot_name *origin">
     <!--joint between {parent} and link_0-->
@@ -168,5 +166,5 @@
       <axis xyz="0 0 1"/>
       <limit lower="${-120 * PI / 180}" upper="${120 * PI / 180}"
-             effort="176" velocity="${150 * PI / 180}" />
+             effort="176" velocity="${75 * PI / 180}" />
       <safety_controller soft_lower_limit="${-118 * PI / 180}"
                          soft_upper_limit="${118 * PI / 180}"

Commit message: Increase the joint safety constraint of urdf

File: iiwas_description/urdf/iiwa14.xacro (robot description, xacro)
@@ -8,5 +8,5 @@
   <xacro:include filename="$(find iiwas_description)/urdf/utilities.xacro" />
   <!-- some constants -->
-  <xacro:property name="safety_controller_k_pos" value="1" />
+  <xacro:property name="safety_controller_k_pos" value="100" />
   <xacro:property name="safety_controller_k_vel" value="10" />
   <xacro:property name="joint_damping" value="0.5" />

Commit message: Update the urdf to stuerz's result, test pinocchio for inertia matrix

File: iiwas_description/urdf/iiwa14.xacro (robot description, xacro)
@@ -57,14 +57,14 @@
                          k_position="${safety_controller_k_pos}"
                          k_velocity="${safety_controller_k_vel}"/>
-      <dynamics damping="${joint_damping}"/>
+      <dynamics damping="0.24150"  friction="0.31909"/>
     </joint>
     <link name="${robot_name}_link_1">
       <inertial>
-        <origin xyz="0 -0.03 0.12" rpy="0 0 0"/>
-<!--        <origin xyz="0.003508 -0.001602 0.171113" rpy="0 0 0"/>  &lt;!&ndash; inertial from sl but in different coordinate system &ndash;&gt;-->
+<!--        <origin xyz="0 -0.03 0.12" rpy="0 0 0"/>-->
+        <origin xyz="-0.003508 0.001602 -0.03139" rpy="0 0 0"/>  <!-- inertial from sl but in different coordinate system -->
         <mass value="3.947808"/>
-<!--        <inertia ixx="0.004554"  ixy="0.000001"  ixz="-0.000002" iyy="0.004542" iyz="0.000005" izz="0.000289" />-->
+        <inertia ixx="0.004554"  ixy="0.00000"  ixz="-0.00000" iyy="0.00454" iyz="0.00001" izz="0.00029" />
 <!--        <inertia ixx="0.4554"  ixy="0.0001"  ixz="-0.0002" iyy="0.4542" iyz="0.0005" izz="0.0289" />-->
-        <inertia ixx="0.1"  ixy="0"  ixz="0" iyy="0.09" iyz="0" izz="0.02" />
+<!--        <inertia ixx="0.1"  ixy="0"  ixz="0" iyy="0.09" iyz="0" izz="0.02" />-->
       </inertial>
       <visual>
@@ -95,14 +95,14 @@
                          k_position="${safety_controller_k_pos}"
                          k_velocity="${safety_controller_k_vel}"/>
-      <dynamics damping="${joint_damping}"/>
+      <dynamics damping="0.37328"  friction="0.18130"/>
     </joint>
     <link name="${robot_name}_link_2">
       <inertial>
-        <origin xyz="0.0003 0.059 0.042" rpy="0 0 0"/>
-<!--        <origin xyz="-0.007671 0.166693  -0.003551" rpy="0 0 0"/>  &lt;!&ndash; inertial from sl but in different coordinate system &ndash;&gt;-->
+<!--        <origin xyz="0.0003 0.059 0.042" rpy="0 0 0"/>-->
+        <origin xyz="-0.007671 0.166693  -0.003551" rpy="0 0 0"/>  <!-- inertial from sl but in different coordinate system -->
         <mass value="4.502752"/>
-<!--        <inertia ixx="0.000318"  ixy="0.000000"  ixz="0.000007" iyy="0.000100" iyz="-0.000003" izz="0.000419" />-->
+        <inertia ixx="0.00032"  ixy="0.00000"  ixz="0.000007" iyy="0.000100" iyz="-0.000003" izz="0.000419" />
 <!--        <inertia ixx="0.0318"  ixy="0.0000"  ixz="0.0007" iyy="0.0100" iyz="-0.0003" izz="0.0419" />-->
-        <inertia ixx="0.05"  ixy="0"  ixz="0" iyy="0.018" iyz="0" izz="0.044" />
+<!--        <inertia ixx="0.05"  ixy="0"  ixz="0" iyy="0.018" iyz="0" izz="0.044" />-->
       </inertial>
       <visual>
@@ -133,14 +133,14 @@
                          k_position="${safety_controller_k_pos}"
                          k_velocity="${safety_controller_k_vel}"/>
-      <dynamics damping="${joint_damping}"/>
+      <dynamics damping="0.11025"  friction="0.07302"/>
     </joint>
     <link name="${robot_name}_link_3">
       <inertial>
-        <origin xyz="0 0.03 0.13" rpy="0 0 0"/>
-<!--        <origin xyz="0.002246 0.034918 0.188978" rpy="0 0 0"/> &lt;!&ndash; inertial from sl but in different coordinate system &ndash;&gt;-->
+<!--        <origin xyz="0 0.03 0.13" rpy="0 0 0"/>-->
+        <origin xyz="-0.002246 -0.034918 -0.02652" rpy="0 0 0"/> <!-- inertial from sl but in different coordinate system -->
         <mass value="2.455197"/>
-<!--        <inertia ixx="0.002233"  ixy="-0.000046"  ixz="0.000068" iyy="0.002191" iyz="0.000072" izz="0.000725" />-->
+        <inertia ixx="0.002233"  ixy="-0.000046"  ixz="0.000068" iyy="0.002191" iyz="0.000072" izz="0.000725" />
 <!--        <inertia ixx="0.2233"  ixy="-0.0046"  ixz="0.0068" iyy="0.2191" iyz="0.0072" izz="0.0725" />-->
-        <inertia ixx="0.08"  ixy="0"  ixz="0" iyy="0.075" iyz="0" izz="0.01" />
+<!--        <inertia ixx="0.08"  ixy="0"  ixz="0" iyy="0.075" iyz="0" izz="0.01" />-->
       </inertial>
       <visual>
@@ -171,14 +171,14 @@
                          k_position="${safety_controller_k_pos}"
                          k_velocity="${safety_controller_k_vel}"/>
-      <dynamics damping="${joint_damping}"/>
+      <dynamics damping="0.10000"  friction="0.17671"/>
     </joint>
     <link name="${robot_name}_link_4">
       <inertial>
-        <origin xyz="0 0.067 0.034" rpy="0 0 0"/>
-<!--        <origin xyz="-0.000196  0.052679 0.038182" rpy="0 0 0"/> &lt;!&ndash; inertial from sl but in different coordinate system &ndash;&gt;-->
+<!--        <origin xyz="0 0.067 0.034" rpy="0 0 0"/>-->
+        <origin xyz="0.000196 -0.052679 0.038182" rpy="0 0 0"/> <!-- inertial from sl but in different coordinate system -->
         <mass value="2.611550"/>
-<!--        <inertia ixx="0.038444"  ixy="0.000880"  ixz="-0.001120" iyy="0.011437" iyz="-0.001113" izz=" 0.049880" />-->
+        <inertia ixx="0.038444"  ixy="0.000880"  ixz="-0.001120" iyy="0.011437" iyz="-0.001113" izz=" 0.049880" />
 <!--        <inertia ixx="3.8444"  ixy="0.0880"  ixz="-0.1120" iyy="1.1437" iyz="-0.1113" izz=" 4.9880" />-->
-        <inertia ixx="0.03"  ixy="0"  ixz="0" iyy="0.01" iyz="0" izz="0.029" />
+<!--        <inertia ixx="0.03"  ixy="0"  ixz="0" iyy="0.01" iyz="0" izz="0.029" />-->
       </inertial>
       <visual>
@@ -209,14 +209,14 @@
                          k_position="${safety_controller_k_pos}"
                          k_velocity="${safety_controller_k_vel}"/>
-      <dynamics damping="${joint_damping}"/>
+      <dynamics damping="0.10000"  friction="0.03463"/>
     </joint>
     <link name="${robot_name}_link_5">
       <inertial>
-        <origin xyz="0.0001 0.021 0.076" rpy="0 0 0"/>
-<!--        <origin xyz="0.000054  -0.002367 0.004164" rpy="0 0 0"/> &lt;!&ndash; inertial from sl but in different coordinate system &ndash;&gt;-->
+<!--        <origin xyz="0.0001 0.021 0.076" rpy="0 0 0"/>-->
+        <origin xyz="0.000054  -0.002367 -0.21134" rpy="0 0 0"/> <!-- inertial from sl but in different coordinate system -->
         <mass value="3.410009"/>
-<!--        <inertia ixx="0.002769"  ixy="-0.000008"  ixz="0.000006" iyy="0.002842" iyz="-0.000001" izz="0.000117" />-->
+        <inertia ixx="0.002769"  ixy="-0.000008"  ixz="0.000006" iyy="0.002842" iyz="-0.000001" izz="0.000117" />
 <!--        <inertia ixx="0.2769"  ixy="-0.0008"  ixz="0.0006" iyy="0.2842" iyz="-0.0001" izz="0.0117" />-->
-        <inertia ixx="0.02"  ixy="0"  ixz="0" iyy="0.018" iyz="0" izz="0.005" />
+<!--        <inertia ixx="0.02"  ixy="0"  ixz="0" iyy="0.018" iyz="0" izz="0.005" />-->
       </inertial>
       <visual>
@@ -247,14 +247,14 @@
                          k_position="${safety_controller_k_pos}"
                          k_velocity="${safety_controller_k_vel}"/>
-      <dynamics damping="${joint_damping}"/>
+      <dynamics damping="0.12484"  friction="0.13391"/>
     </joint>
     <link name="${robot_name}_link_6">
       <inertial>
-        <origin xyz="0 0.0006 0.0004" rpy="0 0 0"/>
-<!--        <origin xyz="0.000492  0.020190  -0.027496" rpy="0 0 0"/>   &lt;!&ndash; inertial from sl but in different coordinate system &ndash;&gt;-->
+<!--        <origin xyz="0 0.0006 0.0004" rpy="0 0 0"/>-->
+        <origin xyz="0.000492  0.020190  -0.027496" rpy="0 0 0"/>   <!-- inertial from sl but in different coordinate system -->
         <mass value="3.387949"/>
-<!--        <inertia ixx="0.000500"  ixy="-0.000050"  ixz="-0.000024" iyy="0.002809" iyz="-0.000041" izz="0.002315" />-->
+        <inertia ixx="0.000500"  ixy="-0.000050"  ixz="-0.000024" iyy="0.002809" iyz="-0.000041" izz="0.002315" />
 <!--        <inertia ixx="0.0500"  ixy="-0.0050"  ixz="-0.0024" iyy="0.2809" iyz="-0.0041" izz="0.2315" />-->
-        <inertia ixx="0.005"  ixy="0"  ixz="0" iyy="0.0036" iyz="0" izz="0.0047" />
+<!--        <inertia ixx="0.005"  ixy="0"  ixz="0" iyy="0.0036" iyz="0" izz="0.0047" />-->
       </inertial>
       <visual>
@@ -285,14 +285,14 @@
                          k_position="${safety_controller_k_pos}"
                          k_velocity="${safety_controller_k_vel}"/>
-      <dynamics damping="${joint_damping}"/>
+      <dynamics damping="0.10000"  friction="0.08710"/>
     </joint>
     <link name="${robot_name}_link_7">
       <inertial>
-        <origin xyz="0 0 0.02" rpy="0 0 0"/>
-<!--        <origin xyz="0.034656 0.023242 -0.009623" rpy="0 0 0"/> &lt;!&ndash; inertial from sl but in different coordinate system &ndash;&gt;-->
+<!--        <origin xyz="0 0 0.02" rpy="0 0 0"/>-->
+        <origin xyz="-0.034656 -0.023242 0.07138" rpy="0 0 0"/> <!-- inertial from sl but in different coordinate system -->
         <mass value="0.354321"/>
-<!--        <inertia ixx="0.007946"  ixy="0.000221"  ixz="-0.000294" iyy=" 0.010889" iyz="-0.000294" izz="0.002944" />-->
+        <inertia ixx="0.007946"  ixy="0.000221"  ixz="-0.000294" iyy=" 0.010889" iyz="-0.000294" izz="0.002944" />
 <!--        <inertia ixx="0.7946"  ixy="0.0221"  ixz="-0.0294" iyy=" 1.0889" iyz="-0.0294" izz="0.2944" />-->
-        <inertia ixx="0.001"  ixy="0"  ixz="0" iyy="0.001" iyz="0" izz="0.001" />
+<!--        <inertia ixx="0.001"  ixy="0"  ixz="0" iyy="0.001" iyz="0" izz="0.001" />-->
       </inertial>
       <visual>
@@ -318,8 +318,8 @@
     <link name="${robot_name}_link_ee">
       <inertial>
-      <origin rpy="0 0 0" xyz="0 0 0.0"/>
-      <mass value="0.0"/>
-      <inertia ixx="0.0" ixy="0.0" ixz="0.0" iyy="0.0" iyz="0.0" izz="0.0"/>
-    </inertial>
+        <origin rpy="0 0 0" xyz="0 0 0.0"/>
+        <mass value="0.0"/>
+        <inertia ixx="0.0" ixy="0.0" ixz="0.0" iyy="0.0" iyz="0.0" izz="0.0"/>
+      </inertial>
     </link>
     <!--Extensions -->

Commit message: Increased inertia and improved gazzebo launch file

File: iiwas_description/urdf/iiwa14.xacro (robot description, xacro)
@@ -64,7 +64,6 @@
         <origin xyz="-0.003508 0.001602 -0.03139" rpy="0 0 0"/>  <!-- inertial from sl but in different coordinate system -->
         <mass value="3.947808"/>
-        <inertia ixx="0.004554"  ixy="0.00000"  ixz="-0.00000" iyy="0.00454" iyz="0.00001" izz="0.00029" />
-<!--        <inertia ixx="0.4554"  ixy="0.0001"  ixz="-0.0002" iyy="0.4542" iyz="0.0005" izz="0.0289" />-->
-<!--        <inertia ixx="0.1"  ixy="0"  ixz="0" iyy="0.09" iyz="0" izz="0.02" />-->
+      <!--    <inertia ixx="0.004554"  ixy="0.00000"  ixz="-0.00000" iyy="0.00454" iyz="0.00001" izz="0.00029" /> -->
+      <inertia ixx="0.4554"  ixy="0.0001"  ixz="-0.0002" iyy="0.4542" iyz="0.0005" izz="0.0289" />
       </inertial>
       <visual>
@@ -102,7 +101,6 @@
         <origin xyz="-0.007671 0.166693  -0.003551" rpy="0 0 0"/>  <!-- inertial from sl but in different coordinate system -->
         <mass value="4.502752"/>
-        <inertia ixx="0.00032"  ixy="0.00000"  ixz="0.000007" iyy="0.000100" iyz="-0.000003" izz="0.000419" />
-<!--        <inertia ixx="0.0318"  ixy="0.0000"  ixz="0.0007" iyy="0.0100" iyz="-0.0003" izz="0.0419" />-->
-<!--        <inertia ixx="0.05"  ixy="0"  ixz="0" iyy="0.018" iyz="0" izz="0.044" />-->
+<!--         <inertia ixx="0.00032"  ixy="0.00000"  ixz="0.000007" iyy="0.000100" iyz="-0.000003" izz="0.000419" /> -->
+       <inertia ixx="0.0318"  ixy="0.0000"  ixz="0.0007" iyy="0.0100" iyz="-0.0003" izz="0.0419" />
       </inertial>
       <visual>
@@ -140,6 +138,6 @@
         <origin xyz="-0.002246 -0.034918 -0.02652" rpy="0 0 0"/> <!-- inertial from sl but in different coordinate system -->
         <mass value="2.455197"/>
-        <inertia ixx="0.002233"  ixy="-0.000046"  ixz="0.000068" iyy="0.002191" iyz="0.000072" izz="0.000725" />
-<!--        <inertia ixx="0.2233"  ixy="-0.0046"  ixz="0.0068" iyy="0.2191" iyz="0.0072" izz="0.0725" />-->
+<!--           <inertia ixx="0.002233"  ixy="-0.000046"  ixz="0.000068" iyy="0.002191" iyz="0.000072" izz="0.000725" /> -->
+        <inertia ixx="0.2233"  ixy="-0.0046"  ixz="0.0068" iyy="0.2191" iyz="0.0072" izz="0.0725" />
 <!--        <inertia ixx="0.08"  ixy="0"  ixz="0" iyy="0.075" iyz="0" izz="0.01" />-->
       </inertial>
@@ -178,7 +176,6 @@
         <origin xyz="0.000196 -0.052679 0.038182" rpy="0 0 0"/> <!-- inertial from sl but in different coordinate system -->
         <mass value="2.611550"/>
-        <inertia ixx="0.038444"  ixy="0.000880"  ixz="-0.001120" iyy="0.011437" iyz="-0.001113" izz=" 0.049880" />
-<!--        <inertia ixx="3.8444"  ixy="0.0880"  ixz="-0.1120" iyy="1.1437" iyz="-0.1113" izz=" 4.9880" />-->
-<!--        <inertia ixx="0.03"  ixy="0"  ixz="0" iyy="0.01" iyz="0" izz="0.029" />-->
+<!--   <inertia ixx="0.038444"  ixy="0.000880"  ixz="-0.001120" iyy="0.011437" iyz="-0.001113" izz=" 0.049880" /> -->
+       <inertia ixx="3.8444"  ixy="0.0880"  ixz="-0.1120" iyy="1.1437" iyz="-0.1113" izz=" 4.9880" />
       </inertial>
       <visual>
@@ -216,7 +213,6 @@
         <origin xyz="0.000054  -0.002367 -0.21134" rpy="0 0 0"/> <!-- inertial from sl but in different coordinate system -->
         <mass value="3.410009"/>
-        <inertia ixx="0.002769"  ixy="-0.000008"  ixz="0.000006" iyy="0.002842" iyz="-0.000001" izz="0.000117" />
-<!--        <inertia ixx="0.2769"  ixy="-0.0008"  ixz="0.0006" iyy="0.2842" iyz="-0.0001" izz="0.0117" />-->
-<!--        <inertia ixx="0.02"  ixy="0"  ixz="0" iyy="0.018" iyz="0" izz="0.005" />-->
+        <!--  <inertia ixx="0.002769"  ixy="-0.000008"  ixz="0.000006" iyy="0.002842" iyz="-0.000001" izz="0.000117" /> -->
+        <inertia ixx="0.2769"  ixy="-0.0008"  ixz="0.0006" iyy="0.2842" iyz="-0.0001" izz="0.0117" />
       </inertial>
       <visual>
@@ -254,7 +250,6 @@
         <origin xyz="0.000492  0.020190  -0.027496" rpy="0 0 0"/>   <!-- inertial from sl but in different coordinate system -->
         <mass value="3.387949"/>
-        <inertia ixx="0.000500"  ixy="-0.000050"  ixz="-0.000024" iyy="0.002809" iyz="-0.000041" izz="0.002315" />
-<!--        <inertia ixx="0.0500"  ixy="-0.0050"  ixz="-0.0024" iyy="0.2809" iyz="-0.0041" izz="0.2315" />-->
-<!--        <inertia ixx="0.005"  ixy="0"  ixz="0" iyy="0.0036" iyz="0" izz="0.0047" />-->
+        <!-- <inertia ixx="0.000500"  ixy="-0.000050"  ixz="-0.000024" iyy="0.002809" iyz="-0.000041" izz="0.002315" /> -->
+        <inertia ixx="0.0500"  ixy="-0.0050"  ixz="-0.0024" iyy="0.2809" iyz="-0.0041" izz="0.2315" />
       </inertial>
       <visual>
@@ -292,7 +287,6 @@
         <origin xyz="-0.034656 -0.023242 0.07138" rpy="0 0 0"/> <!-- inertial from sl but in different coordinate system -->
         <mass value="0.354321"/>
-        <inertia ixx="0.007946"  ixy="0.000221"  ixz="-0.000294" iyy=" 0.010889" iyz="-0.000294" izz="0.002944" />
-<!--        <inertia ixx="0.7946"  ixy="0.0221"  ixz="-0.0294" iyy=" 1.0889" iyz="-0.0294" izz="0.2944" />-->
-<!--        <inertia ixx="0.001"  ixy="0"  ixz="0" iyy="0.001" iyz="0" izz="0.001" />-->
+        <!-- <inertia ixx="0.007946"  ixy="0.000221"  ixz="-0.000294" iyy=" 0.010889" iyz="-0.000294" izz="0.002944" /> -->
+        <inertia ixx="0.7946"  ixy="0.0221"  ixz="-0.0294" iyy=" 1.0889" iyz="-0.0294" izz="0.2944" />
       </inertial>
       <visual>

File: iiwas_description/urdf/iiwas_frame.urdf.xacro (robot description, xacro)
@@ -92,5 +92,5 @@
                 <material name="Brown"/>
             </visual>
-            <collision>
+            <!--  <collision>
                 <origin xyz="0.0 0.0 0.0"
                         rpy="0.0 0.0 0.0"/>
@@ -99,5 +99,5 @@
                 </geometry>
             </collision>
-            <selfCollide>0</selfCollide>
+            <selfCollide>0</selfCollide>  -->
         </link>
         <joint name="back_in" type="fixed">
@@ -159,5 +159,5 @@
                 <material name="Brown"/>
             </visual>
-            <collision>
+            <!-- <collision>
                 <origin xyz="0.0 0.0 0.0"
                         rpy="0.0 0.0 0.0"/>
@@ -166,5 +166,5 @@
                 </geometry>
             </collision>
-            <selfCollide>0</selfCollide>
+            <selfCollide>0</selfCollide>  -->
         </link>
         <joint name="front_out" type="fixed">

Commit message: Test Inertia

File: iiwas_description/urdf/iiwa14.xacro (robot description, xacro)
@@ -64,6 +64,7 @@
         <origin xyz="-0.003508 0.001602 -0.03139" rpy="0 0 0"/>  <!-- inertial from sl but in different coordinate system -->
         <mass value="3.947808"/>
-      <!--    <inertia ixx="0.004554"  ixy="0.00000"  ixz="-0.00000" iyy="0.00454" iyz="0.00001" izz="0.00029" /> -->
-      <inertia ixx="0.4554"  ixy="0.0001"  ixz="-0.0002" iyy="0.4542" iyz="0.0005" izz="0.0289" />
+<!--          <inertia ixx="0.004554"  ixy="0.00000"  ixz="-0.00000" iyy="0.00454" iyz="0.00001" izz="0.00029" />-->
+<!--          <inertia ixx="0.04554"  ixy="0.0000"  ixz="-0.0000" iyy="0.0454" iyz="0.0001" izz="0.0029" />-->
+          <inertia ixx="0.4554"  ixy="0.0001"  ixz="-0.0002" iyy="0.4542" iyz="0.0005" izz="0.0289" />
       </inertial>
       <visual>
@@ -101,6 +102,7 @@
         <origin xyz="-0.007671 0.166693  -0.003551" rpy="0 0 0"/>  <!-- inertial from sl but in different coordinate system -->
         <mass value="4.502752"/>
-<!--         <inertia ixx="0.00032"  ixy="0.00000"  ixz="0.000007" iyy="0.000100" iyz="-0.000003" izz="0.000419" /> -->
-       <inertia ixx="0.0318"  ixy="0.0000"  ixz="0.0007" iyy="0.0100" iyz="-0.0003" izz="0.0419" />
+<!--          <inertia ixx="0.00032"  ixy="0.00000"  ixz="0.000007" iyy="0.000100" iyz="-0.000003" izz="0.000419" />-->
+<!--          <inertia ixx="0.0032"  ixy="0.0000"  ixz="0.00007" iyy="0.00100" iyz="-0.00003" izz="0.00419" />-->
+          <inertia ixx="0.0318"  ixy="0.0000"  ixz="0.0007" iyy="0.0100" iyz="-0.0003" izz="0.0419" />
       </inertial>
       <visual>
@@ -138,7 +140,7 @@
         <origin xyz="-0.002246 -0.034918 -0.02652" rpy="0 0 0"/> <!-- inertial from sl but in different coordinate system -->
         <mass value="2.455197"/>
-<!--           <inertia ixx="0.002233"  ixy="-0.000046"  ixz="0.000068" iyy="0.002191" iyz="0.000072" izz="0.000725" /> -->
-        <inertia ixx="0.2233"  ixy="-0.0046"  ixz="0.0068" iyy="0.2191" iyz="0.0072" izz="0.0725" />
-<!--        <inertia ixx="0.08"  ixy="0"  ixz="0" iyy="0.075" iyz="0" izz="0.01" />-->
+<!--          <inertia ixx="0.002233"  ixy="-0.000046"  ixz="0.000068" iyy="0.002191" iyz="0.000072" izz="0.000725" />-->
+<!--          <inertia ixx="0.02233"  ixy="-0.00046"  ixz="0.00068" iyy="0.02191" iyz="0.00072" izz="0.00725" />-->
+          <inertia ixx="0.2233"  ixy="-0.0046"  ixz="0.0068" iyy="0.2191" iyz="0.0072" izz="0.0725" />
       </inertial>
       <visual>
@@ -176,6 +178,7 @@
         <origin xyz="0.000196 -0.052679 0.038182" rpy="0 0 0"/> <!-- inertial from sl but in different coordinate system -->
         <mass value="2.611550"/>
-<!--   <inertia ixx="0.038444"  ixy="0.000880"  ixz="-0.001120" iyy="0.011437" iyz="-0.001113" izz=" 0.049880" /> -->
-       <inertia ixx="3.8444"  ixy="0.0880"  ixz="-0.1120" iyy="1.1437" iyz="-0.1113" izz=" 4.9880" />
+<!--          <inertia ixx="0.038444"  ixy="0.000880"  ixz="-0.001120" iyy="0.011437" iyz="-0.001113" izz=" 0.049880" />-->
+<!--          <inertia ixx="0.38444"  ixy="0.00880"  ixz="-0.01120" iyy="0.11437" iyz="-0.01113" izz=" 0.49880" />-->
+          <inertia ixx="3.8444"  ixy="0.0880"  ixz="-0.1120" iyy="1.1437" iyz="-0.1113" izz=" 4.9880" />
       </inertial>
       <visual>
@@ -213,6 +216,7 @@
         <origin xyz="0.000054  -0.002367 -0.21134" rpy="0 0 0"/> <!-- inertial from sl but in different coordinate system -->
         <mass value="3.410009"/>
-        <!--  <inertia ixx="0.002769"  ixy="-0.000008"  ixz="0.000006" iyy="0.002842" iyz="-0.000001" izz="0.000117" /> -->
-        <inertia ixx="0.2769"  ixy="-0.0008"  ixz="0.0006" iyy="0.2842" iyz="-0.0001" izz="0.0117" />
+<!--          <inertia ixx="0.002769"  ixy="-0.000008"  ixz="0.000006" iyy="0.002842" iyz="-0.000001" izz="0.000117" />-->
+<!--          <inertia ixx="0.02769"  ixy="-0.00008"  ixz="0.00006" iyy="0.02842" iyz="-0.00001" izz="0.00117" />-->
+          <inertia ixx="0.2769"  ixy="-0.0008"  ixz="0.0006" iyy="0.2842" iyz="-0.0001" izz="0.0117" />
       </inertial>
       <visual>
@@ -250,6 +254,7 @@
         <origin xyz="0.000492  0.020190  -0.027496" rpy="0 0 0"/>   <!-- inertial from sl but in different coordinate system -->
         <mass value="3.387949"/>
-        <!-- <inertia ixx="0.000500"  ixy="-0.000050"  ixz="-0.000024" iyy="0.002809" iyz="-0.000041" izz="0.002315" /> -->
-        <inertia ixx="0.0500"  ixy="-0.0050"  ixz="-0.0024" iyy="0.2809" iyz="-0.0041" izz="0.2315" />
+<!--          <inertia ixx="0.000500"  ixy="-0.000050"  ixz="-0.000024" iyy="0.002809" iyz="-0.000041" izz="0.002315" />-->
+<!--          <inertia ixx="0.00500"  ixy="-0.00050"  ixz="-0.00024" iyy="0.02809" iyz="-0.00041" izz="0.02315" />-->
+          <inertia ixx="0.0500"  ixy="-0.0050"  ixz="-0.0024" iyy="0.2809" iyz="-0.0041" izz="0.2315" />
       </inertial>
       <visual>
@@ -287,6 +292,7 @@
         <origin xyz="-0.034656 -0.023242 0.07138" rpy="0 0 0"/> <!-- inertial from sl but in different coordinate system -->
         <mass value="0.354321"/>
-        <!-- <inertia ixx="0.007946"  ixy="0.000221"  ixz="-0.000294" iyy=" 0.010889" iyz="-0.000294" izz="0.002944" /> -->
-        <inertia ixx="0.7946"  ixy="0.0221"  ixz="-0.0294" iyy=" 1.0889" iyz="-0.0294" izz="0.2944" />
+<!--          <inertia ixx="0.007946"  ixy="0.000221"  ixz="-0.000294" iyy=" 0.010889" iyz="-0.000294" izz="0.002944" />-->
+<!--          <inertia ixx="0.07946"  ixy="0.00221"  ixz="-0.00294" iyy=" 0.10889" iyz="-0.00294" izz="0.02944" />-->
+          <inertia ixx="0.7946"  ixy="0.0221"  ixz="-0.0294" iyy=" 1.0889" iyz="-0.0294" izz="0.2944" />
       </inertial>
       <visual>
