Commit message: Increase the inertia term of the urdf

File: iiwas_description/urdf/iiwa14.xacro (robot description, xacro)
@@ -69,5 +69,6 @@
           <mass value="2.356723"/>
           <origin xyz="0.000000 0.000000 -0.249990" rpy="0 0 0"/>
-          <inertia ixx="0.099939"  ixy="-0.000029"  iyy="0.099716" ixz="-0.000026" iyz="0.000099" izz="0.001000" />
+<!--          <inertia ixx="0.099939"  ixy="-0.000029"  iyy="0.099716" ixz="-0.000026" iyz="0.000099" izz="0.001000" />-->
+          <inertia ixx="0.1"  ixy="0"  ixz="0" iyy="0.1" iyz="0" izz="0.01" />
       </inertial>
       <visual>
@@ -110,5 +111,5 @@
           <mass value="6.000000"/>
           <origin xyz="-0.004595 0.150863 0.028496" rpy="0 0 0"/>
-          <inertia ixx="0.003001"  ixy="-0.000099"  iyy="0.001000" ixz="0.000099" iyz="-0.000099" izz="0.003001" />
+          <inertia ixx="0.030001"  ixy="-0.000999"  iyy="0.010000" ixz="0.000999" iyz="-0.000999" izz="0.030001" />
       </inertial>
       <visual>
@@ -151,5 +152,5 @@
           <mass value="6.00000"/>
           <origin xyz="-0.006630 -0.001947 -0.057071" rpy="0 0 0"/>
-          <inertia ixx="0.003001"  ixy="-0.000099"  iyy="0.003001" ixz="0.000099" iyz="0.000099" izz="0.001000" />
+        <inertia ixx="0.003001"  ixy="-0.000999"  iyy="0.030001" ixz="0.000999" iyz="-0.000999" izz="0.010000" />
       </inertial>
       <visual>

Commit message: Remove the k from ADRC, test the inertia Term

File: iiwas_description/urdf/iiwa14.xacro (robot description, xacro)
@@ -63,6 +63,6 @@
                          k_position="${safety_controller_k_pos}"
                          k_velocity="${safety_controller_k_vel}"/>
-<!--      <dynamics damping="0.24150"  friction="0.31909"/> &lt;!&ndash; ETH &ndash;&gt;-->
-      <dynamics damping="0.330320"  friction="0.384477"/>
+      <dynamics damping="0.24150"  friction="0.31909"/> <!-- ETH -->
+<!--      <dynamics damping="0.330320"  friction="0.384477"/>-->
     </joint>
     <link name="${robot_name}_link_1">
@@ -111,6 +111,6 @@
                          k_position="${safety_controller_k_pos}"
                          k_velocity="${safety_controller_k_vel}"/>
-<!--      <dynamics damping="0.37328"  friction="0.18130"/> &lt;!&ndash; ETH &ndash;&gt;-->
-        <dynamics damping="0.212160"  friction="0.496333"/>
+      <dynamics damping="0.37328"  friction="0.18130"/> <!-- ETH -->
+<!--        <dynamics damping="0.212160"  friction="0.496333"/>-->
     </joint>
     <link name="${robot_name}_link_2">
@@ -159,6 +159,6 @@
                          k_position="${safety_controller_k_pos}"
                          k_velocity="${safety_controller_k_vel}"/>
-<!--      <dynamics damping="0.11025"  friction="0.07302"/> &lt;!&ndash; ETH &ndash;&gt;-->
-        <dynamics damping="0.100000"  friction="0.173951"/>
+      <dynamics damping="0.11025"  friction="0.07302"/> <!-- ETH -->
+<!--        <dynamics damping="0.100000"  friction="0.173951"/>-->
     </joint>
     <link name="${robot_name}_link_3">
@@ -207,6 +207,6 @@
                          k_position="${safety_controller_k_pos}"
                          k_velocity="${safety_controller_k_vel}"/>
-<!--      <dynamics damping="0.10000"  friction="0.17671"/> &lt;!&ndash; ETH &ndash;&gt;-->
-        <dynamics damping="0.219041"  friction="0.375100"/>
+      <dynamics damping="0.10000"  friction="0.17671"/> <!-- ETH -->
+<!--        <dynamics damping="0.219041"  friction="0.375100"/>-->
     </joint>
     <link name="${robot_name}_link_4">
@@ -254,6 +254,6 @@
                          k_position="${safety_controller_k_pos}"
                          k_velocity="${safety_controller_k_vel}"/>
-<!--      <dynamics damping="0.10000"  friction="0.03463"/> &lt;!&ndash; ETH &ndash;&gt;-->
-        <dynamics damping="0.185923"  friction="0.481099"/>
+      <dynamics damping="0.10000"  friction="0.03463"/> <!-- ETH -->
+<!--        <dynamics damping="0.185923"  friction="0.481099"/>-->
     </joint>
     <link name="${robot_name}_link_5">
@@ -301,6 +301,6 @@
                          k_position="${safety_controller_k_pos}"
                          k_velocity="${safety_controller_k_vel}"/>
-<!--      <dynamics damping="0.12484"  friction="0.13391"/> &lt;!&ndash; ETH &ndash;&gt;-->
-        <dynamics damping="0.100000"  friction="0.196149"/>
+      <dynamics damping="0.12484"  friction="0.13391"/> <!-- ETH -->
+<!--        <dynamics damping="0.100000"  friction="0.196149"/>-->
     </joint>
     <link name="${robot_name}_link_6">
@@ -349,6 +349,6 @@
                          k_position="${safety_controller_k_pos}"
                          k_velocity="${safety_controller_k_vel}"/>
-<!--      <dynamics damping="0.10000"  friction="0.08710"/> &lt;!&ndash; ETH &ndash;&gt;-->
-        <dynamics damping="0.100000"  friction="0.299238"/>
+      <dynamics damping="0.10000"  friction="0.08710"/> <!-- ETH -->
+<!--        <dynamics damping="0.100000"  friction="0.05"/>-->
     </joint>
     <link name="${robot_name}_link_7">

Commit message: Modify the urdf of system identification result

File: iiwas_description/urdf/iiwa14.xacro (robot description, xacro)
@@ -63,6 +63,9 @@
                          k_position="${safety_controller_k_pos}"
                          k_velocity="${safety_controller_k_vel}"/>
-      <dynamics damping="0.24150"  friction="0.31909"/> <!-- ETH -->
-<!--      <dynamics damping="0.330320"  friction="0.384477"/>-->
+      <!-- ETH
+      <dynamics damping="0.24150"  friction="0.31909"/>
+      -->
+      <!-- Identified -->
+      <dynamics damping="0.351210"  friction="0.375046"/>
     </joint>
     <link name="${robot_name}_link_1">
@@ -72,9 +75,4 @@
         <mass value="3.947808"/>
         <inertia ixx="0.004554"  ixy="0.00000"  ixz="-0.00000" iyy="0.00454" iyz="0.00001" izz="0.00029" />
-        -->
-        <!-- SysId
-          <mass value="2.356723"/>
-          <origin xyz="0.000000 0.000000 -0.249990" rpy="0 0 0"/>
-          <inertia ixx="0.099939"  ixy="-0.000029"  iyy="0.099716" ixz="-0.000026" iyz="0.000099" izz="0.001000" />
         -->
         <!-- CAD -->
@@ -83,4 +81,9 @@
         <inertia ixx="3.2869e-02" ixy="-4.3000e-07" iyy="3.3168e-02"
                  ixz="9.4000e-07" iyz="4.8970e-03" izz="1.2274e-02"/>
+        <!-- Identified
+        <mass value="4.897254"/>
+        <origin xyz="0.0 0.0 0.0" rpy="0 0 0"/>
+        <inertia ixx="0.000979" ixy="0.0" ixz="0.0" iyy="0.000979" iyz="0.0" izz="0.000945"/>
+         -->
       </inertial>
       <visual>
@@ -111,6 +114,9 @@
                          k_position="${safety_controller_k_pos}"
                          k_velocity="${safety_controller_k_vel}"/>
-      <dynamics damping="0.37328"  friction="0.18130"/> <!-- ETH -->
-<!--        <dynamics damping="0.212160"  friction="0.496333"/>-->
+      <!-- ETH -->
+      <dynamics damping="0.37328"  friction="0.18130"/>
+      <!-- Identified
+      <dynamics damping="0.523418"  friction="0.351184"/>
+      -->
     </joint>
     <link name="${robot_name}_link_2">
@@ -120,9 +126,4 @@
           <origin xyz="-0.007671 0.166693  -0.003551" rpy="0 0 0"/>
           <inertia ixx="0.00032"  ixy="0.00000"  ixz="0.000007" iyy="0.000100" iyz="-0.000003" izz="0.000419" />
-        -->
-        <!-- SysID
-          <mass value="6.000000"/>
-          <origin xyz="-0.004595 0.150863 0.028496" rpy="0 0 0"/>
-          <inertia ixx="0.030001"  ixy="-0.000999"  iyy="0.010000" ixz="0.000999" iyz="-0.000999" izz="0.030001" />
         -->
         <!-- CAD -->
@@ -131,4 +132,9 @@
         <inertia ixx="3.0495e-02" ixy="-3.2800e-05" iyy="1.0969e-02"
                  ixz="2.2370e-05" iyz="4.8615e-03" izz="3.0330e-02"/>
+        <!-- Identified
+        <mass value="4.900332"/>
+        <origin xyz="-0.025248 -0.010544 0.000262" rpy="0 0 0"/>
+        <inertia ixx="0.035650" ixy="-0.010500" ixz="-0.000436" iyy="0.004302" iyz="-0.001409" izz="0.038893"/>
+         -->
       </inertial>
       <visual>
@@ -147,5 +153,5 @@
       </collision>
     </link>
-        <!-- joint between link_2 and link_3 -->
+    <!-- joint between link_2 and link_3 -->
     <joint name="${robot_name}_joint_3" type="revolute">
       <parent link="${robot_name}_link_2"/>
@@ -159,6 +165,9 @@
                          k_position="${safety_controller_k_pos}"
                          k_velocity="${safety_controller_k_vel}"/>
-      <dynamics damping="0.11025"  friction="0.07302"/> <!-- ETH -->
-<!--        <dynamics damping="0.100000"  friction="0.173951"/>-->
+      <!-- ETH -->
+      <dynamics damping="0.11025"  friction="0.07302"/>
+      <!-- Identified
+      <dynamics damping="0.119085"  friction="0.160143"/>
+       -->
     </joint>
     <link name="${robot_name}_link_3">
@@ -168,9 +177,4 @@
         <origin xyz="-0.002246 -0.034918 -0.02652" rpy="0 0 0"/>
         <inertia ixx="0.002233"  ixy="-0.000046"  ixz="0.000068" iyy="0.002191" iyz="0.000072" izz="0.000725" />
-        -->
-        <!-- SysId
-        <mass value="6.00000"/>
-        <origin xyz="-0.006630 -0.001947 -0.057071" rpy="0 0 0"/>
-        <inertia ixx="0.003001"  ixy="-0.000999"  iyy="0.030001" ixz="0.000999" iyz="-0.000999" izz="0.010000" />
         -->
         <!-- CAD -->
@@ -179,4 +183,9 @@
         <inertia ixx="3.1546e-02" ixy="-3.6628e-07" iyy="2.9954e-02"
                  ixz="-3.9154e-07" iyz="-6.1227e-03" izz="9.5594e-03"/>
+        <!-- Identified
+        <mass value="4.832825"/>
+        <origin xyz="0.000148 -0.000314 -0.075932" rpy="0 0 0"/>
+        <inertia ixx="0.021144" ixy="0.000039" ixz="0.002510" iyy="0.021421" iyz="-0.000051" izz="0.001376"/>
+         -->
       </inertial>
       <visual>
@@ -207,6 +216,9 @@
                          k_position="${safety_controller_k_pos}"
                          k_velocity="${safety_controller_k_vel}"/>
-      <dynamics damping="0.10000"  friction="0.17671"/> <!-- ETH -->
-<!--        <dynamics damping="0.219041"  friction="0.375100"/>-->
+      <!-- ETH -->
+      <dynamics damping="0.10000"  friction="0.17671"/>
+      <!-- Identified
+      <dynamics damping="0.501218"  friction="0.206359"/>
+       -->
     </joint>
     <link name="${robot_name}_link_4">
@@ -217,13 +229,14 @@
           <inertia ixx="0.038444"  ixy="0.000880"  ixz="-0.001120" iyy="0.011437" iyz="-0.001113" izz=" 0.049880" />
           -->
-          <!-- SysId
-          <mass value="1.224529"/>
-          <origin xyz="0.044234 0.050000 0.006944" rpy="0 0 0"/>
-          <inertia ixx="0.003001"  ixy="0.000099"  iyy="0.001000" ixz="-0.000099" iyz="0.000099" izz="0.003001" />
+          <!-- CAD -->
+          <mass value="4"/>
+          <origin xyz="-0.000000 0.067480 0.034254" rpy="0 0 0"/>
+          <inertia ixx="2.5087e-02" ixy="-4.3896e-08" iyy="8.9416e-03"
+                   ixz="-1.3169e-07" iyz="4.1448e-03" izz="2.3916e-02" />
+          <!-- Identified
+          <mass value="4.598291"/>
+          <origin xyz="0.006656 0.022481 0.004435" rpy="0 0 0"/>
+          <inertia ixx="0.020475" ixy="0.013639" ixz="-0.00164" iyy="0.011166" iyz="0.002343" izz="0.029962"/>
           -->
-        <mass value="4"/>
-        <origin xyz="-0.000000 0.067480 0.034254" rpy="0 0 0"/>
-        <inertia ixx="2.5087e-02" ixy="-4.3896e-08" iyy="8.9416e-03"
-                 ixz="-1.3169e-07" iyz="4.1448e-03" izz="2.3916e-02" />
       </inertial>
       <visual>
@@ -254,6 +267,9 @@
                          k_position="${safety_controller_k_pos}"
                          k_velocity="${safety_controller_k_vel}"/>
-      <dynamics damping="0.10000"  friction="0.03463"/> <!-- ETH -->
-<!--        <dynamics damping="0.185923"  friction="0.481099"/>-->
+      <!-- ETH -->
+      <dynamics damping="0.10000"  friction="0.03463"/>
+      <!-- Identified
+      <dynamics damping="0.189856"  friction="0.478257"/>
+       -->
     </joint>
     <link name="${robot_name}_link_5">
@@ -264,13 +280,14 @@
         <inertia ixx="0.002769"  ixy="-0.000008"  ixz="0.000006" iyy="0.002842" iyz="-0.000001" izz="0.000117" />
         -->
-        <!-- SysId
-        <mass value="6.00000"/>
-        <origin xyz="-0.002930 0.015256 0.035846" rpy="0 0 0"/>
-        <inertia ixx="0.003001"  ixy="-0.000099"  iyy="0.003001" ixz="-0.000099" iyz="0.000099" izz="0.001000" />
-        -->
+        <!-- CAD -->
         <mass value="3.2"/>
         <origin xyz="0.000125 0.021388 0.075417" rpy="0 0 0"/>
         <inertia ixx="1.9009e-02" ixy="3.3348e-06" iyy="1.6414e-02"
                  ixz="2.9559e-06" iyz="-5.8267e-03" izz="8.4231e-03" />
+        <!-- Identified
+        <mass value="3.873134"/>
+        <origin xyz="0.001058 0.011481 -0.028845" rpy="0 0 0"/>
+        <inertia ixx="0.020982" ixy="0.000060" ixz="-0.000591" iyy="0.020954" iyz="0.000769" izz="0.001127"/>
+         -->
       </inertial>
       <visual>
@@ -301,6 +318,9 @@
                          k_position="${safety_controller_k_pos}"
                          k_velocity="${safety_controller_k_vel}"/>
-      <dynamics damping="0.12484"  friction="0.13391"/> <!-- ETH -->
-<!--        <dynamics damping="0.100000"  friction="0.196149"/>-->
+      <!-- ETH -->
+      <dynamics damping="0.12484"  friction="0.13391"/>
+      <!-- Identified
+      <dynamics damping="0.012774"  friction="0.227769"/>
+       -->
     </joint>
     <link name="${robot_name}_link_6">
@@ -310,9 +330,4 @@
         <origin xyz="0.000492  0.020190  -0.027496" rpy="0 0 0"/>
         <inertia ixx="0.000500"  ixy="-0.000050"  ixz="-0.000024" iyy="0.002809" iyz="-0.000041" izz="0.002315" />
-        -->
-        <!-- SysId
-        <mass value="1.410742"/>
-        <origin xyz="0.015383 -0.046263 0.011131" rpy="0 0 0"/>
-        <inertia ixx="0.001000"  ixy="0.000099"  iyy="0.001000" ixz="0.000099" iyz="0.000099" izz="0.001000" />
         -->
         <!-- CAD -->
@@ -321,4 +336,9 @@
         <inertia ixx="6.1583e-03" ixy="3.4928e-08" iyy="4.4451e-03"
                  ixz="-1.9792e-07" iyz="3.2555e-04" izz="5.7995e-03" />
+        <!-- Identified
+        <mass value="2.556927"/>
+        <origin xyz="0.000874 0.039185 -0.011065" rpy="0 0 0"/>
+        <inertia ixx="0.001284" ixy="0.000057" ixz="-0.000029" iyy="0.001036" iyz="0.000121" izz="0.001177"/>
+         -->
       </inertial>
       <visual>
@@ -349,6 +369,9 @@
                          k_position="${safety_controller_k_pos}"
                          k_velocity="${safety_controller_k_vel}"/>
-      <dynamics damping="0.10000"  friction="0.08710"/> <!-- ETH -->
-<!--        <dynamics damping="0.100000"  friction="0.05"/>-->
+      <!-- ETH -->
+      <dynamics damping="0.10000"  friction="0.08710"/>
+      <!-- Identified
+      <dynamics damping="0.000129"  friction="0.335576"/>
+       -->
     </joint>
     <link name="${robot_name}_link_7">
@@ -358,9 +381,4 @@
         <origin xyz="-0.034656 -0.023242 0.07138" rpy="0 0 0"/>
         <inertia ixx="0.007946"  ixy="0.000221"  ixz="-0.000294" iyy=" 0.010889" iyz="-0.000294" izz="0.002944" />
-        -->
-        <!-- SysId
-        <mass value="1.00000"/>
-        <origin xyz="0.001241 0.004168 0.100000" rpy="0 0 0"/>
-        <inertia ixx="0.001000"  ixy="-0.000099"  iyy="0.001000" ixz="-0.000099" iyz="0.000099" izz="0.001000" />
         -->
         <!-- CAD -->
@@ -369,4 +387,9 @@
         <inertia ixx="3.5211e-04" ixy="-1.4790e-07" iyy="3.5066e-04"
                  ixz="4.7514e-06" iyz="-7.8574e-07" izz="4.3803e-04" />
+        <!-- Identified
+        <mass value="1.554398"/>
+        <origin xyz="-0.000052 -0.000260 -0.067768" rpy="0 0 0"/>
+        <inertia ixx="0.000939" ixy="0.000007" ixz="-0.000015" iyy="0.000936" iyz="0.000008" izz="0.001009"/>
+         -->
       </inertial>
       <visual>

Commit message: Update adrc controller for pybullet simulation
- Increase the safety gain to improve the performance

File: iiwas_description/urdf/iiwa14.xacro (robot description, xacro)
@@ -9,5 +9,5 @@
   <!-- some constants -->
   <xacro:property name="safety_controller_k_pos" value="100" />
-  <xacro:property name="safety_controller_k_vel" value="10" />
+  <xacro:property name="safety_controller_k_vel" value="80" />
   <xacro:property name="joint_damping" value="0.5" />
   <xacro:macro name="iiwa14" params="parent hardware_interface robot_name dynamics_parameter *origin">
@@ -87,5 +87,7 @@
           <origin value="-0.098492 0.000000 0.069462" rpy="0.0 0.0 0.0"/>
           <inertia ixx="0.055704" ixy="0.000000" ixz="0.000356"
-                   iyy="0.056488" iyz="0.000000" izz="0.001462"/>
+                   iyy="0.056488" iyz="0.000000" izz="0.02"/>
+<!--          <inertia ixx="0.055704" ixy="0.000000" ixz="0.000356"-->
+<!--                   iyy="0.056488" iyz="0.000000" izz="0.001462"/>-->
         </xacro:if>
       </inertial>
@@ -191,5 +193,6 @@
           <mass value="2.455197"/>
           <origin xyz="-0.002246 -0.034918 -0.02652" rpy="0 0 0"/>
-          <inertia ixx="0.002233"  ixy="-0.000046"  ixz="0.000068" iyy="0.002191" iyz="0.000072" izz="0.000725" />
+<!--          <inertia ixx="0.002233"  ixy="-0.000046"  ixz="0.000068" iyy="0.002191" iyz="0.000072" izz="0.000725" />-->
+          <inertia ixx="0.002233"  ixy="-0.000046"  ixz="0.000068" iyy="0.002191" iyz="0.000072" izz="0.01" />
         </xacro:if>
         <xacro:if value="${dynamics_parameter == 'cad'}">

Commit message: Fixed the urdf

File: iiwas_description/urdf/iiwa14.xacro (robot description, xacro)
@@ -572,5 +572,5 @@
         <origin xyz="0 0 0" rpy="0 0 0"/>
         <mass value="1e-6"/>
-        <inertia ixx="1"  ixy="0"  ixz="0" iyy="1" iyz="0" izz="1" />
+        <inertia ixx="0.001"  ixy="0"  ixz="0" iyy="0.001" iyz="0" izz="0.001" />
       </inertial>
     </link>
