Commit message: Add iiwas remote launch file
- Add remote launch file and
- refactor joint name
- add flags in ros_control.launch to decide which joint to choose

File: iiwas_description/robots/iiwas_new_frame.urdf (robot description, URDF)
Before this commit: robot iiwas, 27 links, 26 joints
Links:
- link B_link_ee: mass None -> 0.0
- link F_link_ee: mass None -> 0.0
- link back_base: mass None -> 3
- link front_base: mass None -> 3
- link h_bar_back_in: mass None -> 5
- link h_bar_back_out: mass None -> 5
- link h_bar_front_in: mass None -> 5
- link h_bar_front_out: mass None -> 5
- link v_bar_left: mass None -> 8
- link v_bar_right: mass None -> 8
Joints:
- removed joint B_EB
- removed joint B_HR
- removed joint B_SAA
- removed joint B_SFE
- removed joint B_WAA
- removed joint B_WFE
- removed joint B_WR
- removed joint F_EB
- removed joint F_HR
- removed joint F_SAA
- removed joint F_SFE
- removed joint F_WAA
- removed joint F_WFE
- removed joint F_WR
- added joint B_joint_1: type revolute, parent B_link_0, child B_link_1, origin xyz=0 0 0.1575 rpy=0 0 0, axis 0 0 1, limit lower=-2.96705972839 upper=2.96705972839 effort=320 velocity=1.4835298642
- added joint B_joint_2: type revolute, parent B_link_1, child B_link_2, origin xyz=0 0 0.2025 rpy=1.57079632679   0 3.14159265359, axis 0 0 1, limit lower=-2.09439510239 upper=2.09439510239 effort=320 velocity=1.4835298642
- added joint B_joint_3: type revolute, parent B_link_2, child B_link_3, origin xyz=0 0.2045 0 rpy=1.57079632679 0 3.14159265359, axis 0 0 1, limit lower=-2.96705972839 upper=2.96705972839 effort=176 velocity=1.74532925199
- added joint B_joint_4: type revolute, parent B_link_3, child B_link_4, origin xyz=0 0 0.2155 rpy=1.57079632679 0 0, axis 0 0 1, limit lower=-2.09439510239 upper=2.09439510239 effort=176 velocity=1.308996939
- added joint B_joint_5: type revolute, parent B_link_4, child B_link_5, origin xyz=0 0.1845 0 rpy=-1.57079632679 3.14159265359 0, axis 0 0 1, limit lower=-2.96705972839 upper=2.96705972839 effort=110 velocity=2.26892802759
- added joint B_joint_6: type revolute, parent B_link_5, child B_link_6, origin xyz=0 0 0.2155 rpy=1.57079632679 0 0, axis 0 0 1, limit lower=-2.09439510239 upper=2.09439510239 effort=40 velocity=2.35619449019
- added joint B_joint_7: type revolute, parent B_link_6, child B_link_7, origin xyz=0 0.081 0 rpy=-1.57079632679 3.14159265359 0, axis 0 0 1, limit lower=-3.05432619099 upper=3.05432619099 effort=40 velocity=2.35619449019
- added joint F_joint_1: type revolute, parent F_link_0, child F_link_1, origin xyz=0 0 0.1575 rpy=0 0 0, axis 0 0 1, limit lower=-2.96705972839 upper=2.96705972839 effort=320 velocity=1.4835298642
- added joint F_joint_2: type revolute, parent F_link_1, child F_link_2, origin xyz=0 0 0.2025 rpy=1.57079632679   0 3.14159265359, axis 0 0 1, limit lower=-2.09439510239 upper=2.09439510239 effort=320 velocity=1.4835298642
- added joint F_joint_3: type revolute, parent F_link_2, child F_link_3, origin xyz=0 0.2045 0 rpy=1.57079632679 0 3.14159265359, axis 0 0 1, limit lower=-2.96705972839 upper=2.96705972839 effort=176 velocity=1.74532925199
- added joint F_joint_4: type revolute, parent F_link_3, child F_link_4, origin xyz=0 0 0.2155 rpy=1.57079632679 0 0, axis 0 0 1, limit lower=-2.09439510239 upper=2.09439510239 effort=176 velocity=1.308996939
- added joint F_joint_5: type revolute, parent F_link_4, child F_link_5, origin xyz=0 0.1845 0 rpy=-1.57079632679 3.14159265359 0, axis 0 0 1, limit lower=-2.96705972839 upper=2.96705972839 effort=110 velocity=2.26892802759
- added joint F_joint_6: type revolute, parent F_link_5, child F_link_6, origin xyz=0 0 0.2155 rpy=1.57079632679 0 0, axis 0 0 1, limit lower=-2.09439510239 upper=2.09439510239 effort=40 velocity=2.35619449019
- added joint F_joint_7: type revolute, parent F_link_6, child F_link_7, origin xyz=0 0.081 0 rpy=-1.57079632679 3.14159265359 0, axis 0 0 1, limit lower=-3.05432619099 upper=3.05432619099 effort=40 velocity=2.35619449019

File: iiwas_description/urdf/iiwa14.xacro (robot description, xacro)
@@ -48,5 +48,6 @@
     </link>
     <!-- joint between link_0 and link_1 -->
-    <joint name="${robot_name}_SFE" type="revolute">
+    <!--<joint name="${robot_name}_SFE" type="revolute">-->
+    <joint name="${robot_name}_joint_1" type="revolute">
       <parent link="${robot_name}_link_0"/>
       <child link="${robot_name}_link_1"/>
@@ -86,5 +87,6 @@
     </link>
     <!-- joint between link_1 and link_2 -->
-    <joint name="${robot_name}_SAA" type="revolute">
+    <!--<joint name="${robot_name}_SAA" type="revolute">-->
+    <joint name="${robot_name}_joint_2" type="revolute">
       <parent link="${robot_name}_link_1"/>
       <child link="${robot_name}_link_2"/>
@@ -124,5 +126,6 @@
     </link>
     <!-- joint between link_2 and link_3 -->
-    <joint name="${robot_name}_HR" type="revolute">
+    <!--<joint name="${robot_name}_HR" type="revolute">-->
+    <joint name="${robot_name}_joint_3" type="revolute">
       <parent link="${robot_name}_link_2"/>
       <child link="${robot_name}_link_3"/>
@@ -162,5 +165,6 @@
     </link>
     <!-- joint between link_3 and link_4 -->
-    <joint name="${robot_name}_EB" type="revolute">
+    <!--<joint name="${robot_name}_EB" type="revolute">-->
+    <joint name="${robot_name}_joint_4" type="revolute">
       <parent link="${robot_name}_link_3"/>
       <child link="${robot_name}_link_4"/>
@@ -200,5 +204,6 @@
     </link>
     <!-- joint between link_4 and link_5 -->
-    <joint name="${robot_name}_WR" type="revolute">
+    <!--<joint name="${robot_name}_WR" type="revolute">-->
+    <joint name="${robot_name}_joint_5" type="revolute">
       <parent link="${robot_name}_link_4"/>
       <child link="${robot_name}_link_5"/>
@@ -238,5 +243,6 @@
     </link>
     <!-- joint between link_5 and link_6 -->
-    <joint name="${robot_name}_WFE" type="revolute">
+    <!--<joint name="${robot_name}_WFE" type="revolute">-->
+    <joint name="${robot_name}_joint_6" type="revolute">
       <parent link="${robot_name}_link_5"/>
       <child link="${robot_name}_link_6"/>
@@ -276,5 +282,6 @@
     </link>
     <!-- joint between link_6 and link_7 -->
-    <joint name="${robot_name}_WAA" type="revolute">
+    <!--<joint name="${robot_name}_WAA" type="revolute">-->
+    <joint name="${robot_name}_joint_7" type="revolute">
       <parent link="${robot_name}_link_6"/>
       <child link="${robot_name}_link_7"/>

Commit message: Change the frame dependencies
- Robot base is now changable
- Set up new robot positions

File: iiwas_description/robots/iiwas_new_frame.urdf (robot description, URDF)
Before this commit: robot iiwas, 27 links, 26 joints
Joints:
- joint B_joint_1: limit lower=-2.96705972839 upper=2.96705972839 effort=320 velocity=1.4835298642 -> lower=-2.9670597283903604 upper=2.9670597283903604 effort=320 velocity=1.4835298641951802
- joint B_joint_2: limit lower=-2.09439510239 upper=2.09439510239 effort=320 velocity=1.4835298642 -> lower=-2.0943951023931953 upper=2.0943951023931953 effort=320 velocity=1.4835298641951802; origin xyz=0 0 0.2025 rpy=1.57079632679   0 3.14159265359 -> xyz=0 0 0.2025 rpy=1.5707963267948966   0 3.141592653589793
- joint B_joint_3: limit lower=-2.96705972839 upper=2.96705972839 effort=176 velocity=1.74532925199 -> lower=-2.9670597283903604 upper=2.9670597283903604 effort=176 velocity=1.7453292519943295; origin xyz=0 0.2045 0 rpy=1.57079632679 0 3.14159265359 -> xyz=0 0.2045 0 rpy=1.5707963267948966 0 3.141592653589793
- joint B_joint_4: limit lower=-2.09439510239 upper=2.09439510239 effort=176 velocity=1.308996939 -> lower=-2.0943951023931953 upper=2.0943951023931953 effort=176 velocity=1.3089969389957472; origin xyz=0 0 0.2155 rpy=1.57079632679 0 0 -> xyz=0 0 0.2155 rpy=1.5707963267948966 0 0
- joint B_joint_5: limit lower=-2.96705972839 upper=2.96705972839 effort=110 velocity=2.26892802759 -> lower=-2.9670597283903604 upper=2.9670597283903604 effort=110 velocity=2.2689280275926285; origin xyz=0 0.1845 0 rpy=-1.57079632679 3.14159265359 0 -> xyz=0 0.1845 0 rpy=-1.5707963267948966 3.141592653589793 0
- joint B_joint_6: limit lower=-2.09439510239 upper=2.09439510239 effort=40 velocity=2.35619449019 -> lower=-2.0943951023931953 upper=2.0943951023931953 effort=40 velocity=2.356194490192345; origin xyz=0 0 0.2155 rpy=1.57079632679 0 0 -> xyz=0 0 0.2155 rpy=1.5707963267948966 0 0
- joint B_joint_7: limit lower=-3.05432619099 upper=3.05432619099 effort=40 velocity=2.35619449019 -> lower=-3.0543261909900763 upper=3.0543261909900763 effort=40 velocity=2.356194490192345; origin xyz=0 0.081 0 rpy=-1.57079632679 3.14159265359 0 -> xyz=0 0.081 0 rpy=-1.5707963267948966 3.141592653589793 0
- joint F_joint_1: limit lower=-2.96705972839 upper=2.96705972839 effort=320 velocity=1.4835298642 -> lower=-2.9670597283903604 upper=2.9670597283903604 effort=320 velocity=1.4835298641951802
- joint F_joint_2: limit lower=-2.09439510239 upper=2.09439510239 effort=320 velocity=1.4835298642 -> lower=-2.0943951023931953 upper=2.0943951023931953 effort=320 velocity=1.4835298641951802; origin xyz=0 0 0.2025 rpy=1.57079632679   0 3.14159265359 -> xyz=0 0 0.2025 rpy=1.5707963267948966   0 3.141592653589793
- joint F_joint_3: limit lower=-2.96705972839 upper=2.96705972839 effort=176 velocity=1.74532925199 -> lower=-2.9670597283903604 upper=2.9670597283903604 effort=176 velocity=1.7453292519943295; origin xyz=0 0.2045 0 rpy=1.57079632679 0 3.14159265359 -> xyz=0 0.2045 0 rpy=1.5707963267948966 0 3.141592653589793
- joint F_joint_4: limit lower=-2.09439510239 upper=2.09439510239 effort=176 velocity=1.308996939 -> lower=-2.0943951023931953 upper=2.0943951023931953 effort=176 velocity=1.3089969389957472; origin xyz=0 0 0.2155 rpy=1.57079632679 0 0 -> xyz=0 0 0.2155 rpy=1.5707963267948966 0 0
- joint F_joint_5: limit lower=-2.96705972839 upper=2.96705972839 effort=110 velocity=2.26892802759 -> lower=-2.9670597283903604 upper=2.9670597283903604 effort=110 velocity=2.2689280275926285; origin xyz=0 0.1845 0 rpy=-1.57079632679 3.14159265359 0 -> xyz=0 0.1845 0 rpy=-1.5707963267948966 3.141592653589793 0
- joint F_joint_6: limit lower=-2.09439510239 upper=2.09439510239 effort=40 velocity=2.35619449019 -> lower=-2.0943951023931953 upper=2.0943951023931953 effort=40 velocity=2.356194490192345; origin xyz=0 0 0.2155 rpy=1.57079632679 0 0 -> xyz=0 0 0.2155 rpy=1.5707963267948966 0 0
- joint F_joint_7: limit lower=-3.05432619099 upper=3.05432619099 effort=40 velocity=2.35619449019 -> lower=-3.0543261909900763 upper=3.0543261909900763 effort=40 velocity=2.356194490192345; origin xyz=0 0.081 0 rpy=-1.57079632679 3.14159265359 0 -> xyz=0 0.081 0 rpy=-1.5707963267948966 3.141592653589793 0
- joint back_base_B_base_joint: origin xyz=0.0 0.0 0.015 rpy=0.0 0.0 3.14159265359 -> xyz=0.0 0.0 0.015 rpy=0.0 0.0 3.141592653589793
- joint back_in: origin xyz=0.0 0.0 -0.0975 rpy=0.0 0.0 1.57079632679 -> xyz=0.0 0.0 -0.0975 rpy=0.0 0.0 1.5707963267948966
- joint back_out: origin xyz=3.22 0.0 -0.0975 rpy=0.0 0.0 1.57079632679 -> xyz=0.24 0.0 0.0 rpy=0.0 0.0 1.5707963267948966; parent front_base -> back_bar_in
- joint front_in: origin xyz=0.0 0.0 -0.0975 rpy=0.0 0.0 1.57079632679 -> xyz=0.0 0.61 -0.0975 rpy=0.0 0.0 1.5707963267948966
- joint front_out: origin xyz=-0.20 0.0 -0.0975 rpy=0.0 0.0 1.57079632679 -> xyz=-0.20 0.0 0.0 rpy=0.0 0.0 1.5707963267948966; parent front_base -> h_bar_front_in

File: iiwas_description/robots/iiwas_new_frame.urdf.xacro (robot description, xacro)
@@ -7,7 +7,6 @@
     <!-- the mass values and inertia may not be completly correct as the moment so this model should just be used as a kinematic one now-->
     <xacro:property name="M_PI" value="3.1415926535897931"/>
+    <xacro:property name="base_height" default="0.03"/>
     <!-- offset values from world to robot base frame.  0.165+0.015 m is the height of the frame + half height of the plate -->
-    <xacro:property name="base_height" value="0.03"/>
-    <xacro:arg name="front_base_to_back_base_x" default="3.02"/>
     <xacro:arg name="world_to_iiwas_f_x" default="0.0"/>
     <xacro:arg name="world_to_iiwas_f_y" default="0.0"/>
@@ -16,16 +15,14 @@
     <xacro:arg name="world_to_iiwas_f_pitch" default="0.0"/>
     <xacro:arg name="world_to_iiwas_f_yaw" default="0.0"/>
+    <xacro:arg name="world_to_iiwas_b_x" default="0.0"/>
+    <xacro:arg name="world_to_iiwas_b_y" default="0.0"/>
+    <xacro:arg name="world_to_iiwas_b_z" default="0.0"/>
+    <xacro:arg name="world_to_iiwas_b_roll" default="0.0"/>
+    <xacro:arg name="world_to_iiwas_b_pitch" default="0.0"/>
+    <xacro:arg name="world_to_iiwas_b_yaw" default="0.0"/>
     <xacro:arg name="hardware_interface" default="PositionJointInterface"/>
     <!-- construct the iiwas frame, all link is based on the front_base -->
-    <xacro:iiwas_frame name="iiwas_frame">
-        <front>
-            <origin xyz="$(arg world_to_iiwas_f_x) $(arg world_to_iiwas_f_y) ${$(arg world_to_iiwas_f_z) - base_height/2}"
-                    rpy="$(arg world_to_iiwas_f_roll) $(arg world_to_iiwas_f_pitch) $(arg world_to_iiwas_f_yaw)" />
-        </front>
-        <back>
-            <origin xyz="$(arg front_base_to_back_base_x) 0.0 0.0"
-                    rpy="0.0 0.0 0.0" />
-        </back>
-    </xacro:iiwas_frame>
+    <xacro:iiwas_frame name="iiwas_frame" front_x="$(arg world_to_iiwas_f_x)" front_y="$(arg world_to_iiwas_f_y)"
+                        back_x="$(arg world_to_iiwas_b_x)" back_y="$(arg world_to_iiwas_b_y)"/>
     <!-- spawn the robot on each of the base-->
     <!-- iiwas front arm -->

File: iiwas_description/urdf/iiwas_frame.urdf.xacro (robot description, xacro)
@@ -16,8 +16,10 @@
   <xacro:property name="base_w" value="0.35"/>
   <xacro:property name="base_h" value="0.03"/>
-  <xacro:macro name="iiwas_frame" params="name **origin_front **origin_back">
+  <xacro:property name="base_to_bar_y" value="0.61"/>
+  <xacro:macro name="iiwas_frame" params="name front_x front_y back_x back_y">
     <link name="world"/>
     <joint name="front_base_joint" type="fixed">
-      <xacro:insert_block name="origin_front"/>
+      <origin xyz="${front_x} ${front_y} -${base_h/2}"
+            rpy="0.0 0.0 0.0"/>
       <parent link="world"/>
       <child link="front_base"/>
@@ -49,7 +51,40 @@
       <selfCollide>0</selfCollide>
     </link>
+    <joint name="front_in" type="fixed">
+       <origin xyz="0.0 ${-front_y} -${horizontal_bar_inner_h/2 + base_h/2}"
+            rpy="0.0 0.0 0.0"/>
+       <parent link="front_base"/>
+       <child link="h_bar_front_in"/>
+    </joint>
+    <link name="h_bar_front_in">
+      <inertial>
+        <origin xyz="0 0 0" rpy="0 0 0" />
+        <mass value="5" />
+        <inertia
+          ixx="0.0175" ixy="0.0" ixz="0.0"
+          iyy="1.025" iyz="0.0"
+          izz="1.02" />
+      </inertial>
+      <visual>
+        <origin xyz="0.0 0.0 0.0"
+                rpy="0.0 0.0 0.0"/>
+        <geometry>
+          <box size="${horizontal_bar_inner_w} ${horizontal_bar_inner_l} ${horizontal_bar_inner_h}"/>
+        </geometry>
+        <material name="LightGrey"/>
+      </visual>
+      <collision>
+        <origin xyz="0.0 0.0 0.0"
+                rpy="0.0 0.0 0.0"/>
+        <geometry>
+          <box size="${horizontal_bar_inner_w} ${horizontal_bar_inner_l} ${horizontal_bar_inner_h}"/>
+        </geometry>
+      </collision>
+      <selfCollide>0</selfCollide>
+    </link>
     <joint name="back_base_joint" type="fixed">
-      <xacro:insert_block name="origin_back"/>
-      <parent link="front_base"/>
+      <origin xyz="${back_x} ${back_y} -${base_h/2}"
+            rpy="0.0 0.0 0.0"/>
+      <parent link="world"/>
       <child link="back_base"/>
     </joint>
@@ -80,71 +115,7 @@
       <selfCollide>0</selfCollide>
     </link>
-    <joint name="front_in" type="fixed">
-       <origin xyz="0.0 0.0 ${-base_h/2-horizontal_bar_inner_h/2}"
-            rpy="0.0 0.0 ${M_PI/2}"/>
-       <parent link="front_base"/>
-       <child link="h_bar_front_in"/>
-    </joint>
-    <link name="h_bar_front_in">
-      <inertial>
-        <origin xyz="0 0 0" rpy="0 0 0" />
-        <mass value="5" />
-        <inertia
-          ixx="0.0175" ixy="0.0" ixz="0.0"
-          iyy="1.025" iyz="0.0"
-          izz="1.02" />
-      </inertial>
-      <visual>
-        <origin xyz="0.0 0.0 0.0"
-                rpy="0.0 0.0 0.0"/>
-        <geometry>
-          <box size="${horizontal_bar_inner_l} ${horizontal_bar_inner_w} ${horizontal_bar_inner_h}"/>
-        </geometry>
-        <material name="LightGrey"/>
-      </visual>
-      <collision>
-        <origin xyz="0.0 0.0 0.0"
-                rpy="0.0 0.0 0.0"/>
-        <geometry>
-          <box size="${horizontal_bar_inner_l} ${horizontal_bar_inner_w} ${horizontal_bar_inner_h}"/>
-        </geometry>
-      </collision>
-      <selfCollide>0</selfCollide>
-    </link>
-    <joint name="front_out" type="fixed">
-       <origin xyz="-0.20 0.0 ${-base_h/2-horizontal_bar_inner_h/2}"
-            rpy="0.0 0.0 ${M_PI/2}"/>
-       <parent link="front_base"/>
-       <child link="h_bar_front_out"/>
-    </joint>
-    <link name="h_bar_front_out">
-      <inertial>
-        <origin xyz="0 0 0" rpy="0 0 0" />
-        <mass value="5" />
-        <inertia
-          ixx="0.014" ixy="0.0" ixz="0.0"
-          iyy="1.025" iyz="0.0"
-          izz="1.02" />
-      </inertial>
-      <visual>
-        <origin xyz="0.0 0.0 0.0"
-                rpy="0.0 0.0 0.0"/>
-        <geometry>
-          <box size="${horizontal_bar_outer_l} ${horizontal_bar_outer_w} ${horizontal_bar_outer_h}"/>
-        </geometry>
-        <material name="LightGrey"/>
-      </visual>
-      <collision>
-        <origin xyz="0.0 0.0 0.0"
-                rpy="0.0 0.0 0.0"/>
-        <geometry>
-          <box size="${horizontal_bar_outer_l} ${horizontal_bar_outer_w} ${horizontal_bar_outer_h}"/>
-        </geometry>
-      </collision>
-      <selfCollide>0</selfCollide>
-    </link>
     <joint name="back_in" type="fixed">
-       <origin xyz="0.0 0.0 ${-base_h/2-horizontal_bar_inner_h/2}"
-            rpy="0.0 0.0 ${M_PI/2}"/>
+       <origin xyz="0.0 -${back_y} -${horizontal_bar_inner_h/2 + base_h/2}"
+            rpy="0.0 0.0 0.0"/>
        <parent link="back_base"/>
        <child link="h_bar_back_in"/>
@@ -163,24 +134,24 @@
                 rpy="0.0 0.0 0.0"/>
         <geometry>
-          <box size="${horizontal_bar_inner_l} ${horizontal_bar_inner_w} ${horizontal_bar_inner_h}"/>
-        </geometry>
-        <material name="LightGrey"/>
-      </visual>
-      <collision>
-        <origin xyz="0.0 0.0 0.0"
-                rpy="0.0 0.0 0.0"/>
-        <geometry>
-          <box size="${horizontal_bar_inner_l} ${horizontal_bar_inner_w} ${horizontal_bar_inner_h}"/>
-        </geometry>
-      </collision>
-      <selfCollide>0</selfCollide>
-    </link>
-    <joint name="back_out" type="fixed">
-       <origin xyz="3.22 0.0 ${-base_h/2-horizontal_bar_inner_h/2}"
-            rpy="0.0 0.0 ${M_PI/2}"/>
-       <parent link="front_base"/>
-       <child link="h_bar_back_out"/>
-    </joint>
-    <link name="h_bar_back_out">
+          <box size="${horizontal_bar_inner_w} ${horizontal_bar_inner_l} ${horizontal_bar_inner_h}"/>
+        </geometry>
+        <material name="LightGrey"/>
+      </visual>
+      <collision>
+        <origin xyz="0.0 0.0 0.0"
+                rpy="0.0 0.0 0.0"/>
+        <geometry>
+          <box size="${horizontal_bar_inner_w} ${horizontal_bar_inner_l} ${horizontal_bar_inner_h}"/>
+        </geometry>
+      </collision>
+      <selfCollide>0</selfCollide>
+    </link>
+    <joint name="front_out" type="fixed">
+       <origin xyz="0.0 0.0 -${horizontal_bar_outer_h/2 + base_h}"
+            rpy="0.0 0.0 0"/>
+       <parent link="world"/>
+       <child link="h_bar_front_out"/>
+    </joint>
+    <link name="h_bar_front_out">
       <inertial>
         <origin xyz="0 0 0" rpy="0 0 0" />
@@ -195,13 +166,13 @@
                 rpy="0.0 0.0 0.0"/>
         <geometry>
-          <box size="${horizontal_bar_outer_l} ${horizontal_bar_outer_w} ${horizontal_bar_outer_h}"/>
-        </geometry>
-        <material name="LightGrey"/>
-      </visual>
-      <collision>
-        <origin xyz="0.0 0.0 0.0"
-                rpy="0.0 0.0 0.0"/>
-        <geometry>
-          <box size="${horizontal_bar_outer_l} ${horizontal_bar_outer_w} ${horizontal_bar_outer_h}"/>
+          <box size="${horizontal_bar_outer_w} ${horizontal_bar_outer_l} ${horizontal_bar_outer_h}"/>
+        </geometry>
+        <material name="LightGrey"/>
+      </visual>
+      <collision>
+        <origin xyz="0.0 0.0 0.0"
+                rpy="0.0 0.0 0.0"/>
+        <geometry>
+          <box size="${horizontal_bar_outer_w} ${horizontal_bar_outer_l} ${horizontal_bar_outer_h}"/>
         </geometry>
       </collision>
@@ -209,7 +180,7 @@
     </link>
     <joint name="left" type="fixed">
-       <origin xyz="1.51 0.84 ${-base_h/2-horizontal_bar_inner_h/2}"
-            rpy="0.0 0.0 0.0"/>
-       <parent link="front_base"/>
+       <origin xyz="${vertical_bar_l/2 - horizontal_bar_outer_w/2} ${horizontal_bar_outer_l/2 + vertical_bar_w/2} 0.0"
+            rpy="0.0 0.0 ${M_PI}"/>
+       <parent link="h_bar_front_out"/>
        <child link="v_bar_left"/>
     </joint>
@@ -241,7 +212,7 @@
     </link>
     <joint name="frame_right" type="fixed">
-       <origin xyz="1.51 -0.84 ${-base_h/2-horizontal_bar_inner_h / 2.0}"
-            rpy="0.0 0.0 0.0"/>
-       <parent link="front_base"/>
+       <origin xyz="${vertical_bar_l/2 - horizontal_bar_outer_w/2} -${horizontal_bar_outer_l/2 + vertical_bar_w/2} 0.0"
+            rpy="0.0 0.0 0.0"/>
+       <parent link="h_bar_front_out"/>
        <child link="v_bar_right"/>
     </joint>
@@ -268,4 +239,36 @@
         <geometry>
           <box size="${vertical_bar_l} ${vertical_bar_w} ${vertical_bar_h}"/>
+        </geometry>
+      </collision>
+      <selfCollide>0</selfCollide>
+    </link>
+    <joint name="back_out" type="fixed">
+          <origin xyz="${vertical_bar_l/2 - horizontal_bar_outer_w/2} ${horizontal_bar_outer_l/2 + vertical_bar_w/2} 0.0"
+                  rpy="0.0 0.0 0.0"/>
+       <parent link="v_bar_right"/>
+       <child link="h_bar_back_out"/>
+    </joint>
+    <link name="h_bar_back_out">
+      <inertial>
+        <origin xyz="0 0 0" rpy="0 0 0" />
+        <mass value="5" />
+        <inertia
+          ixx="0.014" ixy="0.0" ixz="0.0"
+          iyy="1.025" iyz="0.0"
+          izz="1.02" />
+      </inertial>
+      <visual>
+        <origin xyz="0.0 0.0 0.0"
+                rpy="0.0 0.0 0.0"/>
+        <geometry>
+          <box size="${horizontal_bar_outer_w} ${horizontal_bar_outer_l} ${horizontal_bar_outer_h}"/>
+        </geometry>
+        <material name="LightGrey"/>
+      </visual>
+      <collision>
+        <origin xyz="0.0 0.0 0.0"
+                rpy="0.0 0.0 0.0"/>
+        <geometry>
+          <box size="${horizontal_bar_outer_w} ${horizontal_bar_outer_l} ${horizontal_bar_outer_h}"/>
         </geometry>
       </collision>
