Commit message: change the default value

File: iiwas_description/robots/iiwas_new_frame.urdf (robot description, URDF)
Before this commit: robot iiwas, 27 links, 26 joints
Links:
- link h_bar_back_in: geometry collision box size=0.12 1.56 0.165; visual box size=0.12 1.56 0.165
- link h_bar_back_out: geometry collision box size=0.08 1.56 0.165; visual box size=0.08 1.56 0.165
- link h_bar_front_in: geometry collision box size=0.12 1.56 0.165; visual box size=0.12 1.56 0.165
- link h_bar_front_out: geometry collision box size=0.08 1.56 0.165; visual box size=0.08 1.56 0.165
Joints:
- joint back_base_joint: origin xyz=3.02 0.0 0.0 rpy=0.0 0.0 0.0 -> xyz=3.26 0.61 -0.015 rpy=0.0 0.0 0.0; parent front_base -> world
- joint back_in: origin xyz=0.0 0.0 -0.0975 rpy=0.0 0.0 1.5707963267948966 -> xyz=0.0 -0.61 -0.0975 rpy=0.0 0.0 0.0
- joint back_out: origin xyz=0.24 0.0 0.0 rpy=0.0 0.0 1.5707963267948966 -> xyz=1.71 0.8400000000000001 0.0 rpy=0.0 0.0 0.0; parent back_bar_in -> v_bar_right
- joint frame_right: origin xyz=1.51 -0.84 -0.0975 rpy=0.0 0.0 0.0 -> xyz=1.71 -0.8400000000000001 0.0 rpy=0.0 0.0 0.0; parent front_base -> h_bar_front_out
- joint front_base_joint: origin xyz=0.0 0.0 -0.015 rpy=0.0 0.0 0.0 -> xyz=0.24 -0.61 -0.015 rpy=0.0 0.0 0.0
- joint front_in: origin xyz=0.0 0.61 -0.0975 rpy=0.0 0.0 1.5707963267948966 -> xyz=0.0 0.61 -0.0975 rpy=0.0 0.0 0.0
- joint front_out: origin xyz=-0.20 0.0 0.0 rpy=0.0 0.0 1.5707963267948966 -> xyz=0.0 0.0 -0.1125 rpy=0.0 0.0 0; parent h_bar_front_in -> world
- joint left: origin xyz=1.51 0.84 -0.0975 rpy=0.0 0.0 0.0 -> xyz=1.71 0.8400000000000001 0.0 rpy=0.0 0.0 3.141592653589793; parent front_base -> h_bar_front_out

File: iiwas_description/robots/iiwas_new_frame.urdf.xacro (robot description, xacro)
@@ -9,12 +9,12 @@
     <xacro:property name="base_height" default="0.03"/>
     <!-- offset values from world to robot base frame.  0.165+0.015 m is the height of the frame + half height of the plate -->
-    <xacro:arg name="world_to_iiwas_f_x" default="0.0"/>
-    <xacro:arg name="world_to_iiwas_f_y" default="0.0"/>
+    <xacro:arg name="world_to_iiwas_f_x" default="0.24"/>
+    <xacro:arg name="world_to_iiwas_f_y" default="-0.61"/>
     <xacro:arg name="world_to_iiwas_f_z" default="0.0"/>
     <xacro:arg name="world_to_iiwas_f_roll" default="0.0"/>
     <xacro:arg name="world_to_iiwas_f_pitch" default="0.0"/>
     <xacro:arg name="world_to_iiwas_f_yaw" default="0.0"/>
-    <xacro:arg name="world_to_iiwas_b_x" default="0.0"/>
-    <xacro:arg name="world_to_iiwas_b_y" default="0.0"/>
+    <xacro:arg name="world_to_iiwas_b_x" default="3.26"/>
+    <xacro:arg name="world_to_iiwas_b_y" default="0.61"/>
     <xacro:arg name="world_to_iiwas_b_z" default="0.0"/>
     <xacro:arg name="world_to_iiwas_b_roll" default="0.0"/>
