Commit message: Calibrate the two iiwa robot
- Adjust the urdf to current position

File: iiwas_description/robots/iiwas_new_frame.urdf.xacro (robot description, xacro)
@@ -15,5 +15,5 @@
     <xacro:arg name="world_to_iiwas_f_pitch" default="0.0"/>
     <xacro:arg name="world_to_iiwas_f_yaw" default="0.0"/>
-    <xacro:arg name="world_to_iiwas_b_x" default="3.22"/>
+    <xacro:arg name="world_to_iiwas_b_x" default="3.2"/>
     <xacro:arg name="world_to_iiwas_b_y" default="0.61"/>
     <xacro:arg name="world_to_iiwas_b_z" default="0.0"/>
@@ -24,5 +24,6 @@
     <!-- construct the iiwas frame, all link is based on the front_base -->
     <xacro:iiwas_frame name="iiwas_frame" front_x="$(arg world_to_iiwas_f_x)" front_y="$(arg world_to_iiwas_f_y)"
-                        back_x="$(arg world_to_iiwas_b_x)" back_y="$(arg world_to_iiwas_b_y)"/>
+                       front_z ="$(arg world_to_iiwas_f_z)" back_x="$(arg world_to_iiwas_b_x)"
+                       back_y="$(arg world_to_iiwas_b_y)" back_z ="$(arg world_to_iiwas_b_z)"/>
     <!-- spawn the robot on each of the base-->
     <!-- iiwas front arm -->

File: iiwas_description/urdf/iiwas_frame.urdf.xacro (robot description, xacro)
@@ -19,5 +19,5 @@
     <xacro:property name="world_frame_origin_x" value="-0.048"/>
     <xacro:property name="world_frame_origin_y" value="-0.076"/>
-    <xacro:macro name="iiwas_frame" params="name front_x front_y back_x back_y">
+    <xacro:macro name="iiwas_frame" params="name front_x front_y front_z back_x back_y back_z">
         <link name="world"/>
         <joint name="iiwa_frame_origin_joint" type="fixed">
@@ -65,5 +65,5 @@
             <origin xyz="${front_x - world_frame_origin_x}
                    ${front_y - world_frame_origin_y}
-                   ${base_h/2}"
+                   ${base_h/2 + front_z}"
                     rpy="0.0 0.0 0.0"/>
             <parent link="iiwa_frame_origin"/>
@@ -132,5 +132,5 @@
             <origin xyz="${back_x - world_frame_origin_x}
                      ${back_y - world_frame_origin_y}
-                     ${base_h/2}"
+                     ${base_h/2 + back_z}"
                     rpy="0.0 0.0 0.0"/>
             <parent link="iiwa_frame_origin"/>

Commit message: Clean up the urdf and add inertia of CAD

File: iiwas_description/robots/iiwas_new_frame.urdf.xacro (robot description, xacro)
@@ -6,23 +6,6 @@
     <xacro:property name="M_PI" value="3.1415926535897931"/>
     <xacro:property name="base_height" default="0.03"/>
-    <!-- offset values from world to robot base frame.  0.165+0.015 m is the height of the frame + half height of the plate -->
-    <xacro:arg name="world_to_iiwas_f_x" default="0.190"/>
-    <xacro:arg name="world_to_iiwas_f_y" default="0.813"/>
-    <xacro:arg name="world_to_iiwas_f_z" default="0.0"/>
-    <xacro:arg name="world_to_iiwas_f_roll" default="0.0"/>
-    <xacro:arg name="world_to_iiwas_f_pitch" default="0.0"/>
-    <xacro:arg name="world_to_iiwas_f_yaw" default="0.0"/>
-    <xacro:arg name="world_to_iiwas_b_x" default="3.198"/>
-    <xacro:arg name="world_to_iiwas_b_y" default="0.813"/>
-    <xacro:arg name="world_to_iiwas_b_z" default="0.0"/>
-    <xacro:arg name="world_to_iiwas_b_roll" default="0.0"/>
-    <xacro:arg name="world_to_iiwas_b_pitch" default="0.0"/>
-    <xacro:arg name="world_to_iiwas_b_yaw" default="0.0"/>
     <xacro:arg name="hardware_interface" default="PositionJointInterface"/>
-    <!-- construct the iiwas frame, all link is based on the front_base -->
     <xacro:include filename="$(find iiwas_description)/urdf/iiwas_frame.urdf.xacro"/>
-<!--    <xacro:iiwas_frame name="iiwas_frame" front_x="$(arg world_to_iiwas_f_x)" front_y="$(arg world_to_iiwas_f_y)"-->
-<!--                       front_z ="$(arg world_to_iiwas_f_z)" back_x="$(arg world_to_iiwas_b_x)"-->
-<!--                       back_y="$(arg world_to_iiwas_b_y)" back_z ="$(arg world_to_iiwas_b_z)"/>-->
     <!-- spawn the robot on each of the base-->
     <!-- iiwas front arm -->

File: iiwas_description/urdf/iiwa14.xacro (robot description, xacro)
@@ -20,7 +20,13 @@
     <link name="${robot_name}_link_0">
       <inertial>
+        <!--  Fixed
         <origin xyz="-0.1 0 0.07" rpy="0 0 0"/>
         <mass value="5"/>
         <inertia ixx="0.05"  ixy="0"  ixz="0" iyy="0.06" iyz="0" izz="0.03" />
+        -->
+        <!-- CAD -->
+        <mass value="5.476713"/>
+        <origin xyz="-0.012882 -0.000000 0.071517" rpy="0 0 0"/>
+        <inertia ixx="2.4243e-02"  ixy="2.0000e-08"  iyy="3.0840e-02" ixz="6.7180e-04" iyz="-1.9000e-07" izz="3.3475e-02"/>
       </inertial>
       <visual>
@@ -62,13 +68,19 @@
     <link name="${robot_name}_link_1">
       <inertial>
-          <!-- ETH
-          <origin xyz="-0.003508 0.001602 -0.03139" rpy="0 0 0"/>
-          <mass value="3.947808"/>
-          <inertia ixx="0.004554"  ixy="0.00000"  ixz="-0.00000" iyy="0.00454" iyz="0.00001" izz="0.00029" />
-          -->
+        <!-- ETH
+        <origin xyz="-0.003508 0.001602 -0.03139" rpy="0 0 0"/>
+        <mass value="3.947808"/>
+        <inertia ixx="0.004554"  ixy="0.00000"  ixz="-0.00000" iyy="0.00454" iyz="0.00001" izz="0.00029" />
+        -->
+        <!-- SysId
           <mass value="2.356723"/>
           <origin xyz="0.000000 0.000000 -0.249990" rpy="0 0 0"/>
-<!--          <inertia ixx="0.099939"  ixy="-0.000029"  iyy="0.099716" ixz="-0.000026" iyz="0.000099" izz="0.001000" />-->
-          <inertia ixx="0.1"  ixy="0"  ixz="0" iyy="0.1" iyz="0" izz="0.01" />
+          <inertia ixx="0.099939"  ixy="-0.000029"  iyy="0.099716" ixz="-0.000026" iyz="0.000099" izz="0.001000" />
+        -->
+        <!-- CAD -->
+        <mass value="4.100238"/>
+        <origin xyz="0.000004 -0.033790 0.122349" rpy="0 0 0"/>
+        <inertia ixx="3.2869e-02" ixy="-4.3000e-07" iyy="3.3168e-02"
+                 ixz="9.4000e-07" iyz="4.8970e-03" izz="1.2274e-02"/>
       </inertial>
       <visual>
@@ -104,12 +116,19 @@
     <link name="${robot_name}_link_2">
       <inertial>
-          <!-- ETH
+        <!-- ETH
           <mass value="4.502752"/>
           <origin xyz="-0.007671 0.166693  -0.003551" rpy="0 0 0"/>
           <inertia ixx="0.00032"  ixy="0.00000"  ixz="0.000007" iyy="0.000100" iyz="-0.000003" izz="0.000419" />
-          -->
+        -->
+        <!-- SysID
           <mass value="6.000000"/>
           <origin xyz="-0.004595 0.150863 0.028496" rpy="0 0 0"/>
           <inertia ixx="0.030001"  ixy="-0.000999"  iyy="0.010000" ixz="0.000999" iyz="-0.000999" izz="0.030001" />
+        -->
+        <!-- CAD -->
+        <mass value="3.943457"/>
+        <origin xyz="0.000285 0.058872 0.041961" rpy="0 0 0"/>
+        <inertia ixx="3.0495e-02" ixy="-3.2800e-05" iyy="1.0969e-02"
+                 ixz="2.2370e-05" iyz="4.8615e-03" izz="3.0330e-02"/>
       </inertial>
       <visual>
@@ -128,5 +147,5 @@
       </collision>
     </link>
-    <!-- joint between link_2 and link_3 -->
+        <!-- joint between link_2 and link_3 -->
     <joint name="${robot_name}_joint_3" type="revolute">
       <parent link="${robot_name}_link_2"/>
@@ -145,12 +164,19 @@
     <link name="${robot_name}_link_3">
       <inertial>
-          <!-- ETH
-          <mass value="2.455197"/>
-          <origin xyz="-0.002246 -0.034918 -0.02652" rpy="0 0 0"/>
-          <inertia ixx="0.002233"  ixy="-0.000046"  ixz="0.000068" iyy="0.002191" iyz="0.000072" izz="0.000725" />
-          -->
-          <mass value="6.00000"/>
-          <origin xyz="-0.006630 -0.001947 -0.057071" rpy="0 0 0"/>
+        <!-- ETH
+        <mass value="2.455197"/>
+        <origin xyz="-0.002246 -0.034918 -0.02652" rpy="0 0 0"/>
+        <inertia ixx="0.002233"  ixy="-0.000046"  ixz="0.000068" iyy="0.002191" iyz="0.000072" izz="0.000725" />
+        -->
+        <!-- SysId
+        <mass value="6.00000"/>
+        <origin xyz="-0.006630 -0.001947 -0.057071" rpy="0 0 0"/>
         <inertia ixx="0.003001"  ixy="-0.000999"  iyy="0.030001" ixz="0.000999" iyz="-0.000999" izz="0.010000" />
+        -->
+        <!-- CAD -->
+        <mass value="4"/>
+        <origin xyz="0.000002 0.029546 0.126448" rpy="0 0 0"/>
+        <inertia ixx="3.1546e-02" ixy="-3.6628e-07" iyy="2.9954e-02"
+                 ixz="-3.9154e-07" iyz="-6.1227e-03" izz="9.5594e-03"/>
       </inertial>
       <visual>
@@ -191,7 +217,13 @@
           <inertia ixx="0.038444"  ixy="0.000880"  ixz="-0.001120" iyy="0.011437" iyz="-0.001113" izz=" 0.049880" />
           -->
+          <!-- SysId
           <mass value="1.224529"/>
           <origin xyz="0.044234 0.050000 0.006944" rpy="0 0 0"/>
           <inertia ixx="0.003001"  ixy="0.000099"  iyy="0.001000" ixz="-0.000099" iyz="0.000099" izz="0.003001" />
+          -->
+        <mass value="4"/>
+        <origin xyz="-0.000000 0.067480 0.034254" rpy="0 0 0"/>
+        <inertia ixx="2.5087e-02" ixy="-4.3896e-08" iyy="8.9416e-03"
+                 ixz="-1.3169e-07" iyz="4.1448e-03" izz="2.3916e-02" />
       </inertial>
       <visual>
@@ -227,12 +259,18 @@
     <link name="${robot_name}_link_5">
       <inertial>
-          <!-- ETH
-          <mass value="3.410009"/>
-          <origin xyz="0.000054  -0.002367 -0.21134" rpy="0 0 0"/>
-          <inertia ixx="0.002769"  ixy="-0.000008"  ixz="0.000006" iyy="0.002842" iyz="-0.000001" izz="0.000117" />
-          -->
-          <mass value="6.00000"/>
-          <origin xyz="-0.002930 0.015256 0.035846" rpy="0 0 0"/>
-          <inertia ixx="0.003001"  ixy="-0.000099"  iyy="0.003001" ixz="-0.000099" iyz="0.000099" izz="0.001000" />
+        <!-- ETH
+        <mass value="3.410009"/>
+        <origin xyz="0.000054  -0.002367 -0.21134" rpy="0 0 0"/>
+        <inertia ixx="0.002769"  ixy="-0.000008"  ixz="0.000006" iyy="0.002842" iyz="-0.000001" izz="0.000117" />
+        -->
+        <!-- SysId
+        <mass value="6.00000"/>
+        <origin xyz="-0.002930 0.015256 0.035846" rpy="0 0 0"/>
+        <inertia ixx="0.003001"  ixy="-0.000099"  iyy="0.003001" ixz="-0.000099" iyz="0.000099" izz="0.001000" />
+        -->
+        <mass value="3.2"/>
+        <origin xyz="0.000125 0.021388 0.075417" rpy="0 0 0"/>
+        <inertia ixx="1.9009e-02" ixy="3.3348e-06" iyy="1.6414e-02"
+                 ixz="2.9559e-06" iyz="-5.8267e-03" izz="8.4231e-03" />
       </inertial>
       <visual>
@@ -268,12 +306,19 @@
     <link name="${robot_name}_link_6">
       <inertial>
-          <!-- ETH
-          <mass value="3.387949"/>
-          <origin xyz="0.000492  0.020190  -0.027496" rpy="0 0 0"/>
-          <inertia ixx="0.000500"  ixy="-0.000050"  ixz="-0.000024" iyy="0.002809" iyz="-0.000041" izz="0.002315" />
-          -->
-          <mass value="1.410742"/>
-          <origin xyz="0.015383 -0.046263 0.011131" rpy="0 0 0"/>
-          <inertia ixx="0.001000"  ixy="0.000099"  iyy="0.001000" ixz="0.000099" iyz="0.000099" izz="0.001000" />
+        <!-- ETH
+        <mass value="3.387949"/>
+        <origin xyz="0.000492  0.020190  -0.027496" rpy="0 0 0"/>
+        <inertia ixx="0.000500"  ixy="-0.000050"  ixz="-0.000024" iyy="0.002809" iyz="-0.000041" izz="0.002315" />
+        -->
+        <!-- SysId
+        <mass value="1.410742"/>
+        <origin xyz="0.015383 -0.046263 0.011131" rpy="0 0 0"/>
+        <inertia ixx="0.001000"  ixy="0.000099"  iyy="0.001000" ixz="0.000099" iyz="0.000099" izz="0.001000" />
+        -->
+        <!-- CAD -->
+        <mass value="2.2"/>
+        <origin xyz="-0.000000 0.002431 -0.001270" rpy="0 0 0"/>
+        <inertia ixx="6.1583e-03" ixy="3.4928e-08" iyy="4.4451e-03"
+                 ixz="-1.9792e-07" iyz="3.2555e-04" izz="5.7995e-03" />
       </inertial>
       <visual>
@@ -309,12 +354,19 @@
     <link name="${robot_name}_link_7">
       <inertial>
-          <!-- ETH
-          <mass value="0.354321"/>
-          <origin xyz="-0.034656 -0.023242 0.07138" rpy="0 0 0"/>
-          <inertia ixx="0.007946"  ixy="0.000221"  ixz="-0.000294" iyy=" 0.010889" iyz="-0.000294" izz="0.002944" />
-          -->
-          <mass value="1.00000"/>
-          <origin xyz="0.001241 0.004168 0.100000" rpy="0 0 0"/>
-          <inertia ixx="0.001000"  ixy="-0.000099"  iyy="0.001000" ixz="-0.000099" iyz="0.000099" izz="0.001000" />
+        <!-- ETH
+        <mass value="0.354321"/>
+        <origin xyz="-0.034656 -0.023242 0.07138" rpy="0 0 0"/>
+        <inertia ixx="0.007946"  ixy="0.000221"  ixz="-0.000294" iyy=" 0.010889" iyz="-0.000294" izz="0.002944" />
+        -->
+        <!-- SysId
+        <mass value="1.00000"/>
+        <origin xyz="0.001241 0.004168 0.100000" rpy="0 0 0"/>
+        <inertia ixx="0.001000"  ixy="-0.000099"  iyy="0.001000" ixz="-0.000099" iyz="0.000099" izz="0.001000" />
+        -->
+        <!-- CAD -->
+        <mass value="0.4"/>
+        <origin xyz="0.000540 0.000569 0.026582" rpy="0 0 0"/>
+        <inertia ixx="3.5211e-04" ixy="-1.4790e-07" iyy="3.5066e-04"
+                 ixz="4.7514e-06" iyz="-7.8574e-07" izz="4.3803e-04" />
       </inertial>
       <visual>
