Commit message: Separate the description into two namespaces
- Separate robot description into iiwas_frame iiwa_front iiwa_back namespace

File: iiwas_description/robots/iiwa.urdf.xacro (robot description, xacro)
@@ -2,16 +2,23 @@
 <robot name="iiwa14" xmlns:xacro="http://www.ros.org/wiki/xacro">
   <!-- Import Rviz colors -->
-  <xacro:include filename="$(find iiwa_description)/urdf/materials.xacro" />
+  <xacro:include filename="$(find iiwas_description)/urdf/materials.xacro" />
   <!--Import the lbr iiwa macro -->
-  <xacro:include filename="$(find iiwa_description)/urdf/iiwa14.xacro"/>
+  <xacro:include filename="$(find iiwas_description)/urdf/iiwa14.xacro"/>
+  <xacro:property name="base_height" default="0.03"/>
   <xacro:arg name="hardware_interface" default="PositionJointInterface"/>
-  <xacro:arg name="robot_name" default="iiwa"/>
-  <xacro:arg name="origin_xyz" default="0 0 0"/>
-  <xacro:arg name="origin_rpy" default="0 0 0"/>
+  <xacro:arg name="robot_name" default="F"/>
+  <xacro:arg name="parent" default="front_base"/>
+  <xacro:arg name="base_rpy" default="0 0 0"/>
+  <xacro:arg name="namespace" default=""/>
   <!-- Fix to world just for testing -->
-  <link name="world"/>
+  <link name="$(arg parent)"/>
   <!--iiwa-->
-  <xacro:iiwa14 hardware_interface="$(arg hardware_interface)" robot_name="$(arg robot_name)" parent="world">
-    <origin xyz="$(arg origin_xyz)" rpy="$(arg origin_rpy)" />
+  <xacro:iiwa14 hardware_interface="$(arg hardware_interface)" robot_name="$(arg robot_name)" parent="$(arg parent)">
+    <origin xyz="0 0 ${base_height/2}" rpy="$(arg base_rpy)" />
   </xacro:iiwa14>
+  <gazebo>
+    <plugin name="gazebo_ros_control" filename="libgazebo_ros_control.so">
+      <robotParam>$(arg namespace)/robot_description</robotParam>
+    </plugin>
+  </gazebo>
 </robot>

File: iiwas_description/robots/iiwas_new_frame.urdf.xacro (robot description, xacro)
@@ -2,5 +2,5 @@
 <robot name="iiwas" xmlns:xacro="http://www.ros.org/wiki/xacro">
     <xacro:include filename="$(find iiwas_description)/urdf/materials.xacro" />
-    <xacro:include filename="$(find iiwas_description)/urdf/iiwas_frame.urdf.xacro"/>
+    <xacro:include filename="$(find iiwas_description)/urdf/iiwas_frame.xacro"/>
     <xacro:include filename="$(find iiwas_description)/urdf/iiwa14.xacro"/>
     <xacro:include filename="$(find iiwas_description)/urdf/util_defs.xml"/>

File: iiwas_description/urdf/iiwas_frame.xacro (robot description, xacro)
@@ -291,8 +291,13 @@
             <selfCollide>0</selfCollide>
         </link>
-        <gazebo reference="${name}">
-            <material value="Gazebo/Black"/>
-            <turnGravityOff>0
-            </turnGravityOff> <!-- use gravity for the base even if disabled for the arms in order to prevent iiwas from falling-->
+        <gazebo reference="front_base_joint">
+            <preserveFixedJoint>true</preserveFixedJoint>
+        </gazebo>
+        <gazebo reference="front_base">
+        </gazebo>
+        <gazebo reference="back_base_joint">
+            <preserveFixedJoint>true</preserveFixedJoint>
+        </gazebo>
+        <gazebo reference="back_base">
         </gazebo>
     </xacro:macro>

Commit message: Add namespace for two separate robots description
- Test joint_trajectory_controller

File: iiwas_description/robots/iiwa.urdf.xacro (robot description, xacro)
@@ -10,5 +10,4 @@
   <xacro:arg name="parent" default="front_base"/>
   <xacro:arg name="base_rpy" default="0 0 0"/>
-  <xacro:arg name="namespace" default=""/>
   <!-- Fix to world just for testing -->
   <link name="$(arg parent)"/>
@@ -17,7 +16,9 @@
     <origin xyz="0 0 ${base_height/2}" rpy="$(arg base_rpy)" />
   </xacro:iiwa14>
+  <gazebo reference="$(arg parent)">
+    <kinematic>true</kinematic>
+  </gazebo>
   <gazebo>
     <plugin name="gazebo_ros_control" filename="libgazebo_ros_control.so">
-      <robotParam>$(arg namespace)/robot_description</robotParam>
     </plugin>
   </gazebo>

File: iiwas_description/robots/iiwas_frame_urdf.xacro (robot description, xacro)
@@ -1,7 +1,6 @@
 <?xml version="1.0"?>
-<robot name="iiwas" xmlns:xacro="http://www.ros.org/wiki/xacro">
+<robot name="iiwas_frame" xmlns:xacro="http://www.ros.org/wiki/xacro">
     <xacro:include filename="$(find iiwas_description)/urdf/materials.xacro" />
     <xacro:include filename="$(find iiwas_description)/urdf/iiwas_frame.xacro"/>
-    <xacro:arg name="namespace" default="/iiwas_frame"/>
     <xacro:property name="M_PI" value="3.1415926535897931"/>
     <xacro:arg name="world_to_front_base_x" default="0.190"/>
@@ -17,12 +16,5 @@
     <gazebo>
         <plugin name="gazebo_ros_control" filename="libgazebo_ros_control.so">
-            <robotParam>$(arg namespace)/robot_description</robotParam>
         </plugin>
     </gazebo>
-<!--    <gazebo reference="iiwas_frame">-->
-<!--        <material value="Gazebo/Black"/>-->
-<!--        <static>true</static>-->
-<!--        <turnGravityOff>0-->
-<!--        </turnGravityOff> &lt;!&ndash; use gravity for the base even if disabled for the arms in order to prevent iiwas from falling&ndash;&gt;-->
-<!--    </gazebo>-->
 </robot>

File: iiwas_description/urdf/iiwas_frame.xacro (robot description, xacro)
@@ -133,5 +133,5 @@
                      ${back_y - world_frame_origin_y}
                      ${base_h/2 + back_z}"
-                    rpy="0.0 0.0 0.0"/>
+                    rpy="0.0 0.0 ${M_PI}"/>
             <parent link="iiwa_frame_origin"/>
             <child link="back_base"/>

Commit message: Work on iiwa robot urdf
- added setter for robot position
- removed useless parameter
- by default, fixed to world

File: iiwas_description/robots/iiwa.urdf.xacro (robot description, xacro)
@@ -5,8 +5,8 @@
   <!--Import the lbr iiwa macro -->
   <xacro:include filename="$(find iiwas_description)/urdf/iiwa14.xacro"/>
-  <xacro:property name="base_height" default="0.03"/>
   <xacro:arg name="hardware_interface" default="PositionJointInterface"/>
   <xacro:arg name="robot_name" default="F"/>
-  <xacro:arg name="parent" default="front_base"/>
+  <xacro:arg name="parent" default="world"/>
+  <xacro:arg name="base_xyz" default="0 0 0"/>
   <xacro:arg name="base_rpy" default="0 0 0"/>
   <!-- Fix to world just for testing -->
@@ -14,9 +14,6 @@
   <!--iiwa-->
   <xacro:iiwa14 hardware_interface="$(arg hardware_interface)" robot_name="$(arg robot_name)" parent="$(arg parent)">
-    <origin xyz="0 0 ${base_height/2}" rpy="$(arg base_rpy)" />
+    <origin xyz="$(arg base_xyz)" rpy="$(arg base_rpy)" />
   </xacro:iiwa14>
-  <gazebo reference="$(arg parent)">
-    <kinematic>true</kinematic>
-  </gazebo>
   <gazebo>
     <plugin name="gazebo_ros_control" filename="libgazebo_ros_control.so">
